Commit message: update urdf

File: simple_model.urdf (robot description, URDF)
Before this commit: robot simple_box, 17 links, 16 joints
Links:
- link base_link: geometry collision box size=0.2 0.1 0.1; visual box size=0.2 0.14 0.12
- link head: geometry collision box size=0.1 0.1 0.1; visual box size=0.15 0.1 0.1
Joints:
- joint armLU_to_armLL: limit lower=-1.57 upper=0 effort=10 velocity=1.0 -> lower=-1.2 upper=-0.2 effort=10 velocity=1.0
- joint armRU_to_armRL: limit lower=-1.57 upper=0 effort=10 velocity=1.0 -> lower=-1.2 upper=-0.2 effort=10 velocity=1.0
- joint base_to_armLU: limit lower=0 upper=1.57 effort=10 velocity=1.0 -> lower=0.6 upper=1.57 effort=10 velocity=1.0; origin xyz=0.05 -0.1 0 rpy=0 0 0 -> xyz=0.05 -0.095 0 rpy=0 0 0
- joint base_to_armRU: limit lower=0 upper=1.57 effort=10 velocity=1.0 -> lower=0.6 upper=1.57 effort=10 velocity=1.0; origin xyz=0.05 0.1 0 rpy=0 0 0 -> xyz=0.05 0.095 0 rpy=0 0 0
- joint base_to_legBaseL: limit lower=-1.57 upper=1.57 effort=10 velocity=1.0 -> lower=-0.785398 upper=0.785398 effort=10 velocity=1.0; origin xyz=-0.05 -0.05 -0.06 rpy=0 0 0 -> xyz=-0.05 -0.045 -0.06 rpy=0 0 0
- joint base_to_legBaseR: limit lower=-1.57 upper=1.57 effort=10 velocity=1.0 -> lower=-0.785398 upper=0.785398 effort=10 velocity=1.0; origin xyz=-0.05 0.05 -0.06 rpy=0 0 0 -> xyz=-0.05 0.045 -0.06 rpy=0 0 0
- joint base_to_neckBottom: limit lower=-1.57 upper=1.57 effort=10 velocity=1.0 -> lower=-1 upper=1 effort=10 velocity=1.0
- joint legBaseL_to_legHutoL: limit lower=-1.57 upper=1.57 effort=10 velocity=1.0 -> lower=-1.57 upper=0.75 effort=10 velocity=1.0
- joint legBaseR_to_legHutoR: limit lower=-1.57 upper=1.57 effort=10 velocity=1.0 -> lower=-1.57 upper=0.75 effort=10 velocity=1.0
- joint legHutoL_to_legSuneL: limit lower=-1.57 upper=1.57 effort=10 velocity=1.0 -> lower=0.2 upper=1.6 effort=10 velocity=1.0
- joint legHutoR_to_legSuneR: limit lower=-1.57 upper=1.57 effort=10 velocity=1.0 -> lower=0.2 upper=1.6 effort=10 velocity=1.0
- joint legSuneL_to_footL: limit lower=-1.57 upper=1.57 effort=10 velocity=1.0 -> lower=-1.7 upper=-0.2 effort=10 velocity=1.0
- joint legSuneR_to_footR: limit lower=-1.57 upper=1.57 effort=10 velocity=1.0 -> lower=-1.7 upper=-0.2 effort=10 velocity=1.0
- joint neckBottom_to_neckMid: limit lower=-1.57 upper=1.57 effort=10 velocity=1.0 -> lower=-1 upper=1 effort=10 velocity=1.0
- joint neckMid_to_neckTop: limit lower=-1.57 upper=1.57 effort=10 velocity=1.0 -> lower=-0.6 upper=0.75 effort=10 velocity=1.0
- joint neckTop_to_head: limit lower=-1 upper=1 effort=10 velocity=1.0 -> lower=-0.5 upper=0.5 effort=10 velocity=1.0

Commit message: trained

File: simple_model.urdf (robot description, URDF)
Before this commit: robot simple_box, 17 links, 16 joints
Links:
- link armLL: mass 1.0 -> 0.2
- link armLU: mass 1.0 -> 0.2
- link armRL: mass 1.0 -> 0.2
- link armRU: mass 1.0 -> 0.2
- link footL: mass 1.0 -> 0.3
- link footR: mass 1.0 -> 0.3
- link head: mass 1.0 -> 0.5
- link legBaseL: mass 1.0 -> 0.3
- link legBaseR: mass 1.0 -> 0.3
- link legHutoL: mass 1.0 -> 0.3
- link legHutoR: mass 1.0 -> 0.3
- link legSuneL: mass 1.0 -> 0.3
- link legSuneR: mass 1.0 -> 0.3
- link neckBottom: mass 1.0 -> 0.2
- link neckMid: mass 1.0 -> 0.2
- link neckTop: mass 1.0 -> 0.2
Joints:
- joint legHutoL_to_legSuneL: limit lower=0.2 upper=1.6 effort=10 velocity=1.0 -> lower=0.2 upper=1.8 effort=10 velocity=1.0
- joint legHutoR_to_legSuneR: limit lower=0.2 upper=1.6 effort=10 velocity=1.0 -> lower=0.2 upper=1.8 effort=10 velocity=1.0
- joint legSuneL_to_footL: limit lower=-1.7 upper=-0.2 effort=10 velocity=1.0 -> lower=-2.5 upper=-0.2 effort=10 velocity=1.0
- joint legSuneR_to_footR: limit lower=-1.7 upper=-0.2 effort=10 velocity=1.0 -> lower=-2.5 upper=-0.2 effort=10 velocity=1.0
