Commit message: Set motor baudrate to 115200 and add update utility script

File: animatronics_urdf_description/animatronics_urdf_description_standalone.urdf (robot description, URDF)
Before this commit: robot animatronics_urdf, 54 links, 53 joints
Links:
- link 2XC_430_v6_1: geometry collision mesh filename=meshes/2XC-430_v6_1.stl scale=0.001 0.001 0.001; visual mesh filename=meshes/2XC-430_v6_1.stl scale=0.001 0.001 0.001
- link Adafruit_BNO055_STEMMA_QT_v1_1: geometry collision mesh filename=meshes/Adafruit_BNO055_STEMMA_QT_v1_1.stl scale=0.001 0.001 0.001; visual mesh filename=meshes/Adafruit_BNO055_STEMMA_QT_v1_1.stl scale=0.001 0.001 0.001
- link Adafruit_BNO055_STEMMA_QT_v1_2: geometry collision mesh filename=meshes/Adafruit_BNO055_STEMMA_QT_v1_2.stl scale=0.001 0.001 0.001; visual mesh filename=meshes/Adafruit_BNO055_STEMMA_QT_v1_2.stl scale=0.001 0.001 0.001
- link Adafruit_BNO055_STEMMA_QT_v1_3: geometry collision mesh filename=meshes/Adafruit_BNO055_STEMMA_QT_v1_3.stl scale=0.001 0.001 0.001; visual mesh filename=meshes/Adafruit_BNO055_STEMMA_QT_v1_3.stl scale=0.001 0.001 0.001
- link AxisNeckL_v13_1: geometry collision mesh filename=meshes/AxisNeckL_v13_1.stl scale=0.001 0.001 0.001; visual mesh filename=meshes/AxisNeckL_v13_1.stl scale=0.001 0.001 0.001
- link AxisNeckR_v10_1: geometry collision mesh filename=meshes/AxisNeckR_v10_1.stl scale=0.001 0.001 0.001; visual mesh filename=meshes/AxisNeckR_v10_1.stl scale=0.001 0.001 0.001
- link GearNeck_v10_1: geometry collision mesh filename=meshes/GearNeck_v10_1.stl scale=0.001 0.001 0.001; visual mesh filename=meshes/GearNeck_v10_1.stl scale=0.001 0.001 0.001
- link GearNeck_v10_2: geometry collision mesh filename=meshes/GearNeck_v10_2.stl scale=0.001 0.001 0.001; visual mesh filename=meshes/GearNeck_v10_2.stl scale=0.001 0.001 0.001
- link HeadJoint2_v6_1: geometry collision mesh filename=meshes/HeadJoint2_v6_1.stl scale=0.001 0.001 0.001; visual mesh filename=meshes/HeadJoint2_v6_1.stl scale=0.001 0.001 0.001
- link HeadMainPlate_v4_1: geometry collision mesh filename=meshes/HeadMainPlate_v4_1.stl scale=0.001 0.001 0.001; visual mesh filename=meshes/HeadMainPlate_v4_1.stl scale=0.001 0.001 0.001
- link Jaw_v4_1: geometry collision mesh filename=meshes/Jaw_v4_1.stl scale=0.001 0.001 0.001; visual mesh filename=meshes/Jaw_v4_1.stl scale=0.001 0.001 0.001
- link LegA_v14_1: geometry collision mesh filename=meshes/LegA_v14_1.stl scale=0.001 0.001 0.001; visual mesh filename=meshes/LegA_v14_1.stl scale=0.001 0.001 0.001
- link LegA_v14_2: geometry collision mesh filename=meshes/LegA_v14_2.stl scale=0.001 0.001 0.001; visual mesh filename=meshes/LegA_v14_2.stl scale=0.001 0.001 0.001
- link LegBone_v20_1: geometry collision mesh filename=meshes/LegBone_v20_1.stl scale=0.001 0.001 0.001; visual mesh filename=meshes/LegBone_v20_1.stl scale=0.001 0.001 0.001
- link LegBone_v20_2: geometry collision mesh filename=meshes/LegBone_v20_2.stl scale=0.001 0.001 0.001; visual mesh filename=meshes/LegBone_v20_2.stl scale=0.001 0.001 0.001
- link LegBone_v20_3: geometry collision mesh filename=meshes/LegBone_v20_3.stl scale=0.001 0.001 0.001; visual mesh filename=meshes/LegBone_v20_3.stl scale=0.001 0.001 0.001
- link LegBone_v20_4: geometry collision mesh filename=meshes/LegBone_v20_4.stl scale=0.001 0.001 0.001; visual mesh filename=meshes/LegBone_v20_4.stl scale=0.001 0.001 0.001
- link LegEndCover_v6_1: geometry collision mesh filename=meshes/LegEndCover_v6_1.stl scale=0.001 0.001 0.001; visual mesh filename=meshes/LegEndCover_v6_1.stl scale=0.001 0.001 0.001
- link LegEndCover_v6_2: geometry collision mesh filename=meshes/LegEndCover_v6_2.stl scale=0.001 0.001 0.001; visual mesh filename=meshes/LegEndCover_v6_2.stl scale=0.001 0.001 0.001
- link LegEnd_v9_1: geometry collision mesh filename=meshes/LegEnd_v9_1.stl scale=0.001 0.001 0.001; visual mesh filename=meshes/LegEnd_v9_1.stl scale=0.001 0.001 0.001
- link LegEnd_v9_2: geometry collision mesh filename=meshes/LegEnd_v9_2.stl scale=0.001 0.001 0.001; visual mesh filename=meshes/LegEnd_v9_2.stl scale=0.001 0.001 0.001
- link LegRotatorB_v6_1: geometry collision mesh filename=meshes/LegRotatorB_v6_1.stl scale=0.001 0.001 0.001; visual mesh filename=meshes/LegRotatorB_v6_1.stl scale=0.001 0.001 0.001
- link LegRotatorB_v6_2: geometry collision mesh filename=meshes/LegRotatorB_v6_2.stl scale=0.001 0.001 0.001; visual mesh filename=meshes/LegRotatorB_v6_2.stl scale=0.001 0.001 0.001
- link LegRotator_v6_1: geometry collision mesh filename=meshes/LegRotator_v6_1.stl scale=0.001 0.001 0.001; visual mesh filename=meshes/LegRotator_v6_1.stl scale=0.001 0.001 0.001
- link LegRotator_v6_2: geometry collision mesh filename=meshes/LegRotator_v6_2.stl scale=0.001 0.001 0.001; visual mesh filename=meshes/LegRotator_v6_2.stl scale=0.001 0.001 0.001
- link LegSupport_v23_1: geometry collision mesh filename=meshes/LegSupport_v23_1.stl scale=0.001 0.001 0.001; visual mesh filename=meshes/LegSupport_v23_1.stl scale=0.001 0.001 0.001
- link Neck2body_v96_1: geometry collision mesh filename=meshes/Neck2body_v96_1.stl scale=0.001 0.001 0.001; visual mesh filename=meshes/Neck2body_v96_1.stl scale=0.001 0.001 0.001
- link NeckJointH_v23_1: geometry collision mesh filename=meshes/NeckJointH_v23_1.stl scale=0.001 0.001 0.001; visual mesh filename=meshes/NeckJointH_v23_1.stl scale=0.001 0.001 0.001
- link NeckMidGearAxis_v6_1: geometry collision mesh filename=meshes/NeckMidGearAxis_v6_1.stl scale=0.001 0.001 0.001; visual mesh filename=meshes/NeckMidGearAxis_v6_1.stl scale=0.001 0.001 0.001
- link NeckMidGearB_v13_1: geometry collision mesh filename=meshes/NeckMidGearB_v13_1.stl scale=0.001 0.001 0.001; visual mesh filename=meshes/NeckMidGearB_v13_1.stl scale=0.001 0.001 0.001
- link NeckMidGearHolder_v6_1: geometry collision mesh filename=meshes/NeckMidGearHolder_v6_1.stl scale=0.001 0.001 0.001; visual mesh filename=meshes/NeckMidGearHolder_v6_1.stl scale=0.001 0.001 0.001
- link NeckTop_v17_1: geometry collision mesh filename=meshes/NeckTop_v17_1.stl scale=0.001 0.001 0.001; visual mesh filename=meshes/NeckTop_v17_1.stl scale=0.001 0.001 0.001
- link RASPBERRY_PI_5_cooler_v2_v4_1: geometry collision mesh filename=meshes/RASPBERRY_PI_5+cooler_v2_v4_1.stl scale=0.001 0.001 0.001; visual mesh filename=meshes/RASPBERRY_PI_5+cooler_v2_v4_1.stl scale=0.001 0.001 0.001
- link XL_430_new_v5_1: geometry collision mesh filename=meshes/XL-430_new_v5_1.stl scale=0.001 0.001 0.001; visual mesh filename=meshes/XL-430_new_v5_1.stl scale=0.001 0.001 0.001
- link XL_430_new_v5_2: geometry collision mesh filename=meshes/XL-430_new_v5_2.stl scale=0.001 0.001 0.001; visual mesh filename=meshes/XL-430_new_v5_2.stl scale=0.001 0.001 0.001
- link XL_430_new_v5_3: geometry collision mesh filename=meshes/XL-430_new_v5_3.stl scale=0.001 0.001 0.001; visual mesh filename=meshes/XL-430_new_v5_3.stl scale=0.001 0.001 0.001
- link XL_430_new_v5_5: geometry collision mesh filename=meshes/XL-430_new_v5_5.stl scale=0.001 0.001 0.001; visual mesh filename=meshes/XL-430_new_v5_5.stl scale=0.001 0.001 0.001
- link XL_430_new_v5_6: geometry collision mesh filename=meshes/XL-430_new_v5_6.stl scale=0.001 0.001 0.001; visual mesh filename=meshes/XL-430_new_v5_6.stl scale=0.001 0.001 0.001
- link XL_430_new_v5_7: geometry collision mesh filename=meshes/XL-430_new_v5_7.stl scale=0.001 0.001 0.001; visual mesh filename=meshes/XL-430_new_v5_7.stl scale=0.001 0.001 0.001
- link XL_430_new_v5_8: geometry collision mesh filename=meshes/XL-430_new_v5_8.stl scale=0.001 0.001 0.001; visual mesh filename=meshes/XL-430_new_v5_8.stl scale=0.001 0.001 0.001
- link XM_H_D_540_N101_I101_v3_1: geometry collision mesh filename=meshes/XM,H,D-540.N101.I101_v3_1.stl scale=0.001 0.001 0.001; visual mesh filename=meshes/XM,H,D-540.N101.I101_v3_1.stl scale=0.001 0.001 0.001
- link XM_H_D_540_N101_I101_v3_10: geometry collision mesh filename=meshes/XM,H,D-540.N101.I101_v3_10.stl scale=0.001 0.001 0.001; visual mesh filename=meshes/XM,H,D-540.N101.I101_v3_10.stl scale=0.001 0.001 0.001
- link XM_H_D_540_N101_I101_v3_2: geometry collision mesh filename=meshes/XM,H,D-540.N101.I101_v3_2.stl scale=0.001 0.001 0.001; visual mesh filename=meshes/XM,H,D-540.N101.I101_v3_2.stl scale=0.001 0.001 0.001
- link XM_H_D_540_N101_I101_v3_3: geometry collision mesh filename=meshes/XM,H,D-540.N101.I101_v3_3.stl scale=0.001 0.001 0.001; visual mesh filename=meshes/XM,H,D-540.N101.I101_v3_3.stl scale=0.001 0.001 0.001
- link XM_H_D_540_N101_I101_v3_4: geometry collision mesh filename=meshes/XM,H,D-540.N101.I101_v3_4.stl scale=0.001 0.001 0.001; visual mesh filename=meshes/XM,H,D-540.N101.I101_v3_4.stl scale=0.001 0.001 0.001
- link XM_H_D_540_N101_I101_v3_5: geometry collision mesh filename=meshes/XM,H,D-540.N101.I101_v3_5.stl scale=0.001 0.001 0.001; visual mesh filename=meshes/XM,H,D-540.N101.I101_v3_5.stl scale=0.001 0.001 0.001
- link XM_H_D_540_N101_I101_v3_6: geometry collision mesh filename=meshes/XM,H,D-540.N101.I101_v3_6.stl scale=0.001 0.001 0.001; visual mesh filename=meshes/XM,H,D-540.N101.I101_v3_6.stl scale=0.001 0.001 0.001
- link XM_H_D_540_N101_I101_v3_7: geometry collision mesh filename=meshes/XM,H,D-540.N101.I101_v3_7.stl scale=0.001 0.001 0.001; visual mesh filename=meshes/XM,H,D-540.N101.I101_v3_7.stl scale=0.001 0.001 0.001
- link XM_H_D_540_N101_I101_v3_8: geometry collision mesh filename=meshes/XM,H,D-540.N101.I101_v3_8.stl scale=0.001 0.001 0.001; visual mesh filename=meshes/XM,H,D-540.N101.I101_v3_8.stl scale=0.001 0.001 0.001
- link XM_H_D_540_N101_I101_v3_9: geometry collision mesh filename=meshes/XM,H,D-540.N101.I101_v3_9.stl scale=0.001 0.001 0.001; visual mesh filename=meshes/XM,H,D-540.N101.I101_v3_9.stl scale=0.001 0.001 0.001
- link base_link: geometry collision mesh filename=meshes/base_link.stl scale=0.001 0.001 0.001; visual mesh filename=meshes/base_link.stl scale=0.001 0.001 0.001

Commit message: Set motor effort limits to 10Nm in URDF and simulator

File: animatronics_urdf_description/animatronics_urdf_description_standalone.urdf (robot description, URDF)
Before this commit: robot animatronics_urdf, 54 links, 53 joints
Joints:
- joint Revolute_10: limit lower=-1.570796 upper=0.0 effort=100 velocity=100 -> lower=-1.570796 upper=0.0 effort=10.0 velocity=100
- joint Revolute_11: limit lower=0.0 upper=1.570796 effort=100 velocity=100 -> lower=0.0 upper=1.570796 effort=10.0 velocity=100
- joint Revolute_14: limit lower=-0.698132 upper=0.872665 effort=100 velocity=100 -> lower=-0.698132 upper=0.872665 effort=10.0 velocity=100
- joint Revolute_15: limit lower=-0.872665 upper=0.698132 effort=100 velocity=100 -> lower=-0.872665 upper=0.698132 effort=10.0 velocity=100
- joint Revolute_18: limit lower=-1.570796 upper=0.0 effort=100 velocity=100 -> lower=-1.570796 upper=0.0 effort=10.0 velocity=100
- joint Revolute_19: limit lower=0.0 upper=1.570796 effort=100 velocity=100 -> lower=0.0 upper=1.570796 effort=10.0 velocity=100
- joint Revolute_22: limit lower=-1.570796 upper=0.0 effort=100 velocity=100 -> lower=-1.570796 upper=0.0 effort=10.0 velocity=100
- joint Revolute_23: limit lower=0.0 upper=1.570796 effort=100 velocity=100 -> lower=0.0 upper=1.570796 effort=10.0 velocity=100
- joint Revolute_40: limit lower=-1.396263 upper=0.349066 effort=100 velocity=100 -> lower=-1.396263 upper=0.349066 effort=10.0 velocity=100
- joint Revolute_42: limit lower=-1.570796 upper=1.570796 effort=100 velocity=100 -> lower=-1.570796 upper=1.570796 effort=10.0 velocity=100
- joint Revolute_50: limit lower=-1.308997 upper=0.0 effort=100 velocity=100 -> lower=-1.308997 upper=0.0 effort=10.0 velocity=100
