Commit message: update robot urdf and meshes

File: animatronics_urdf_description/animatronics_urdf_description_standalone.urdf (robot description, URDF)
Before this commit: robot animatronics_urdf, 54 links, 53 joints
Links:
- removed link 2XC_430_v6_1
- removed link Adafruit_BNO055_STEMMA_QT_v1_1
- removed link Adafruit_BNO055_STEMMA_QT_v1_2
- removed link Adafruit_BNO055_STEMMA_QT_v1_3
- removed link AxisNeckL_v13_1
- removed link AxisNeckR_v10_1
- removed link GearNeck_v10_1
- removed link GearNeck_v10_2
- removed link HeadJoint2_v6_1
- removed link HeadMainPlate_v4_1
- removed link LegA_v14_1
- removed link LegA_v14_2
- removed link LegBone_v20_1
- removed link LegBone_v20_2
- removed link LegBone_v20_3
- removed link LegBone_v20_4
- removed link LegEndCover_v6_1
- removed link LegEndCover_v6_2
- removed link LegEnd_v9_1
- removed link LegEnd_v9_2
- removed link LegRotatorB_v6_1
- removed link LegRotatorB_v6_2
- removed link LegRotator_v6_1
- removed link LegRotator_v6_2
- removed link LegSupport_v23_1
- removed link Neck2body_v96_1
- removed link NeckJointH_v23_1
- removed link NeckMidGearAxis_v6_1
- removed link NeckMidGearB_v13_1
- removed link NeckMidGearHolder_v6_1
- removed link NeckTop_v17_1
- removed link RASPBERRY_PI_5_cooler_v2_v4_1
- removed link XL_430_new_v5_1
- removed link XL_430_new_v5_2
- removed link XL_430_new_v5_3
- removed link XL_430_new_v5_5
- removed link XL_430_new_v5_6
- removed link XL_430_new_v5_7
- removed link XL_430_new_v5_8
- removed link XM_H_D_540_N101_I101_v3_1
- removed link XM_H_D_540_N101_I101_v3_10
- removed link XM_H_D_540_N101_I101_v3_2
- removed link XM_H_D_540_N101_I101_v3_3
- removed link XM_H_D_540_N101_I101_v3_4
- removed link XM_H_D_540_N101_I101_v3_5
- removed link XM_H_D_540_N101_I101_v3_6
- removed link XM_H_D_540_N101_I101_v3_7
- removed link XM_H_D_540_N101_I101_v3_8
- removed link XM_H_D_540_N101_I101_v3_9
- removed link imu_link 1
- removed link imu_link 2
- removed link imu_link 3
- added link 2XC-430_v6_1, mass 0.09031899704975468; collision mesh filename=package://animatronics_urdf_description/meshes/2XC-430_v6_1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 scale=0.001 0.001 0.001; visual mesh filename=package://animatronics_urdf_description/meshes/2XC-430_v6_1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 scale=0.001 0.001 0.001
- added link 51202_v2_1, mass 0.05505680395324213; collision mesh filename=package://animatronics_urdf_description/meshes/51202_v2_1.s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 scale=0.001 0.001 0.001; visual mesh filename=package://animatronics_urdf_description/meshes/51202_v2_1.s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 scale=0.001 0.001 0.001
- added link 51202_v2_2, mass 0.05505680395324213; collision mesh filename=package://animatronics_urdf_description/meshes/51202_v2_2.s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 scale=0.001 0.001 0.001; visual mesh filename=package://animatronics_urdf_description/meshes/51202_v2_2.s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 scale=0.001 0.001 0.001
- added link 51202_v2_3, mass 0.05505680395324213; collision mesh filename=package://animatronics_urdf_description/meshes/51202_v2_3.s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 scale=0.001 0.001 0.001; visual mesh filename=package://animatronics_urdf_description/meshes/51202_v2_3.s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 scale=0.001 0.001 0.001
- added link 51202_v2_4, mass 0.05505680395324213; collision mesh filename=package://animatronics_urdf_description/meshes/51202_v2_4.s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 scale=0.001 0.001 0.001; visual mesh filename=package://animatronics_urdf_description/meshes/51202_v2_4.s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 scale=0.001 0.001 0.001
- added link 6900ZZNR_v2_1, mass 0.014205025342471455; collision mesh filename=package://animatronics_urdf_description/meshes/6900ZZNR_v2_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 scale=0.001 0.001 0.001; visual mesh filename=package://animatronics_urdf_description/meshes/6900ZZNR_v2_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 scale=0.001 0.001 0.001
- added link 6900ZZNR_v2_2, mass 0.014205025342471455; collision mesh filename=package://animatronics_urdf_description/meshes/6900ZZNR_v2_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 scale=0.001 0.001 0.001; visual mesh filename=package://animatronics_urdf_description/meshes/6900ZZNR_v2_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 scale=0.001 0.001 0.001
- added link Head_Joint_v6_1, mass 0.01706262563442855; collision mesh filename=package://animatronics_urdf_description/meshes/Head_Joint_v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 scale=0.001 0.001 0.001; visual mesh filename=package://animatronics_urdf_description/meshes/Head_Joint_v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 scale=0.001 0.001 0.001
- added link Head_MainPlate_v4_1, mass 0.4432124636647733; collision mesh filename=package://animatronics_urdf_description/meshes/Head_MainPla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 scale=0.001 0.001 0.001; visual mesh filename=package://animatronics_urdf_description/meshes/Head_MainPla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 scale=0.001 0.001 0.001
- added link Leg01_v11_1, mass 0.244537289734516; collision mesh filename=package://animatronics_urdf_description/meshes/Leg01_v11_1.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 scale=0.001 0.001 0.001; visual mesh filename=package://animatronics_urdf_description/meshes/Leg01_v11_1.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 scale=0.001 0.001 0.001
- added link Leg01_v11_2, mass 0.244537289734516; collision mesh filename=package://animatronics_urdf_description/meshes/Leg01_v11_2.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 scale=0.001 0.001 0.001; visual mesh filename=package://animatronics_urdf_description/meshes/Leg01_v11_2.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 scale=0.001 0.001 0.001
- added link Leg02_v10_1, mass 0.7208590729525296; collision mesh filename=package://animatronics_urdf_description/meshes/Leg02_v10_1.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 scale=0.001 0.001 0.001; visual mesh filename=package://animatronics_urdf_description/meshes/Leg02_v10_1.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 scale=0.001 0.001 0.001
- added link Leg02_v10_2, mass 0.7208590729525296; collision mesh filename=package://animatronics_urdf_description/meshes/Leg02_v10_2.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 scale=0.001 0.001 0.001; visual mesh filename=package://animatronics_urdf_description/meshes/Leg02_v10_2.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 scale=0.001 0.001 0.001
- added link Leg03_v28_1, mass 0.0705061968864148; collision mesh filename=package://animatronics_urdf_description/meshes/Leg03_v28_1.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 scale=0.001 0.001 0.001; visual mesh filename=package://animatronics_urdf_description/meshes/Leg03_v28_1.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 scale=0.001 0.001 0.001
- added link Leg03_v28_2, mass 0.0705061968864148; collision mesh filename=package://animatronics_urdf_description/meshes/Leg03_v28_2.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 scale=0.001 0.001 0.001; visual mesh filename=package://animatronics_urdf_description/meshes/Leg03_v28_2.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 scale=0.001 0.001 0.001
- added link Leg04_v11_1, mass 1.201075021531332; collision mesh filename=package://animatronics_urdf_description/meshes/Leg04_v11_1.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 scale=0.001 0.001 0.001; visual mesh filename=package://animatronics_urdf_description/meshes/Leg04_v11_1.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 scale=0.001 0.001 0.001
- added link Leg04_v11_2, mass 1.201075021531332; collision mesh filename=package://animatronics_urdf_description/meshes/Leg04_v11_2.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 scale=0.001 0.001 0.001; visual mesh filename=package://animatronics_urdf_description/meshes/Leg04_v11_2.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 scale=0.001 0.001 0.001
- added link Leg_Cover_v3_1, mass 0.15624009364552216; collision mesh filename=package://animatronics_urdf_description/meshes/Leg_Cover_v3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 scale=0.001 0.001 0.001; visual mesh filename=package://animatronics_urdf_description/meshes/Leg_Cover_v3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 scale=0.001 0.001 0.001
- added link Leg_Cover_v3_2, mass 0.15624009364552216; collision mesh filename=package://animatronics_urdf_description/meshes/Leg_Cover_v3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 scale=0.001 0.001 0.001; visual mesh filename=package://animatronics_urdf_description/meshes/Leg_Cover_v3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 scale=0.001 0.001 0.001
- added link Leg_Rotator_v10_1, mass 0.17090794364421608; collision mesh filename=package://animatronics_urdf_description/meshes/Leg_Rotator_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 scale=0.001 0.001 0.001; visual mesh filename=package://animatronics_urdf_description/meshes/Leg_Rotator_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 scale=0.001 0.001 0.001
- added link Leg_Rotator_v10_2, mass 0.17090794364421608; collision mesh filename=package://animatronics_urdf_description/meshes/Leg_Rotator_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 scale=0.001 0.001 0.001; visual mesh filename=package://animatronics_urdf_description/meshes/Leg_Rotator_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 scale=0.001 0.001 0.001
- added link NeckMidGearHolder_v1_1, mass 0.063161529786995; collision mesh filename=package://animatronics_urdf_description/meshes/NeckMidGearH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 scale=0.001 0.001 0.001; visual mesh filename=package://animatronics_urdf_description/meshes/NeckMidGearH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 scale=0.001 0.001 0.001
- added link Neck_Bar_v1_1, mass 0.022635141245255556; collision mesh filename=package://animatronics_urdf_description/meshes/Neck_Bar_v1_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 scale=0.001 0.001 0.001; visual mesh filename=package://animatronics_urdf_description/meshes/Neck_Bar_v1_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 scale=0.001 0.001 0.001
- added link Neck_Bar_v1_2, mass 0.022635141245255556; collision mesh filename=package://animatronics_urdf_description/meshes/Neck_Bar_v1_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 scale=0.001 0.001 0.001; visual mesh filename=package://animatronics_urdf_description/meshes/Neck_Bar_v1_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 scale=0.001 0.001 0.001
- added link Neck_Gear_Mid_Axis_v6_1, mass 0.02076155413049806; collision mesh filename=package://animatronics_urdf_description/meshes/Neck_Gear_Mi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 scale=0.001 0.001 0.001; visual mesh filename=package://animatronics_urdf_description/meshes/Neck_Gear_Mi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 scale=0.001 0.001 0.001
- added link Neck_Gear_Mid_v13_1, mass 0.14220453425486923; collision mesh filename=package://animatronics_urdf_description/meshes/Neck_Gear_Mi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 scale=0.001 0.001 0.001; visual mesh filename=package://animatronics_urdf_description/meshes/Neck_Gear_Mi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 scale=0.001 0.001 0.001
- added link Neck_Gear_Top_v17_1, mass 0.325166045089014; collision mesh filename=package://animatronics_urdf_description/meshes/Neck_Gear_To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 scale=0.001 0.001 0.001; visual mesh filename=package://animatronics_urdf_description/meshes/Neck_Gear_To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 scale=0.001 0.001 0.001
- added link Neck_Gear_v10_1, mass 0.014297337764134846; collision mesh filename=package://animatronics_urdf_description/meshes/Neck_Gear_v1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 scale=0.001 0.001 0.001; visual mesh filename=package://animatronics_urdf_description/meshes/Neck_Gear_v1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 scale=0.001 0.001 0.001
- added link Neck_JointH_v28_1, mass 0.4802070004701405; collision mesh filename=package://animatronics_urdf_description/meshes/Neck_JointH_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 scale=0.001 0.001 0.001; visual mesh filename=package://animatronics_urdf_description/meshes/Neck_JointH_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 scale=0.001 0.001 0.001
- added link Tail_Base_v3_1, mass 1.3964434577559302; collision mesh filename=package://animatronics_urdf_description/meshes/Tail_Base_v3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 scale=0.001 0.001 0.001; visual mesh filename=package://animatronics_urdf_description/meshes/Tail_Base_v3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 scale=0.001 0.001 0.001
- added link XL-430_new_v5_1, mass 0.33677880262575866; collision mesh filename=package://animatronics_urdf_description/meshes/XL-430_new_v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 scale=0.001 0.001 0.001; visual mesh filename=package://animatronics_urdf_description/meshes/XL-430_new_v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 scale=0.001 0.001 0.001
- added link XL-430_new_v5_2, mass 0.33677880262575866; collision mesh filename=package://animatronics_urdf_description/meshes/XL-430_new_v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 scale=0.001 0.001 0.001; visual mesh filename=package://animatronics_urdf_description/meshes/XL-430_new_v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 scale=0.001 0.001 0.001
- added link XM,H,D-540.N101.I101_v5_1, mass 0.6640277986148612; collision mesh filename=package://animatronics_urdf_description/meshes/XM,H,D-540.N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 scale=0.001 0.001 0.001; visual mesh filename=package://animatronics_urdf_description/meshes/XM,H,D-540.N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 scale=0.001 0.001 0.001
- added link XM,H,D-540.N101.I101_v5_2, mass 0.6640277986148612; collision mesh filename=package://animatronics_urdf_description/meshes/XM,H,D-540.N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 scale=0.001 0.001 0.001; visual mesh filename=package://animatronics_urdf_description/meshes/XM,H,D-540.N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 scale=0.001 0.001 0.001
- added link XM,H,D-540.N101.I101_v5_3, mass 0.6640277986148612; collision mesh filename=package://animatronics_urdf_description/meshes/XM,H,D-540.N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 scale=0.001 0.001 0.001; visual mesh filename=package://animatronics_urdf_description/meshes/XM,H,D-540.N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 scale=0.001 0.001 0.001
- added link XM,H,D-540.N101.I101_v5_4, mass 0.6640277986148612; collision mesh filename=package://animatronics_urdf_description/meshes/XM,H,D-540.N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 scale=0.001 0.001 0.001; visual mesh filename=package://animatronics_urdf_description/meshes/XM,H,D-540.N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 scale=0.001 0.001 0.001
- added link XM,H,D-540.N101.I101_v5_5, mass 0.6640277986148612; collision mesh filename=package://animatronics_urdf_description/meshes/XM,H,D-540.N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 scale=0.001 0.001 0.001; visual mesh filename=package://animatronics_urdf_description/meshes/XM,H,D-540.N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 scale=0.001 0.001 0.001
- added link XM,H,D-540.N101.I101_v5_6, mass 0.6640277986148612; collision mesh filename=package://animatronics_urdf_description/meshes/XM,H,D-540.N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 scale=0.001 0.001 0.001; visual mesh filename=package://animatronics_urdf_description/meshes/XM,H,D-540.N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 scale=0.001 0.001 0.001
- added link XM,H,D-540.N101.I101_v5_7, mass 0.6640277986148612; collision mesh filename=package://animatronics_urdf_description/meshes/XM,H,D-540.N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 scale=0.001 0.001 0.001; visual mesh filename=package://animatronics_urdf_description/meshes/XM,H,D-540.N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 scale=0.001 0.001 0.001
- added link XM,H,D-540.N101.I101_v5_8, mass 0.6640277986148612; collision mesh filename=package://animatronics_urdf_description/meshes/XM,H,D-540.N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 scale=0.001 0.001 0.001; visual mesh filename=package://animatronics_urdf_description/meshes/XM,H,D-540.N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 scale=0.001 0.001 0.001
- added link XM,H-430_idler_v3_1, mass 0.12871928366116375; collision mesh filename=package://animatronics_urdf_description/meshes/XM,H-430_idl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 scale=0.001 0.001 0.001; visual mesh filename=package://animatronics_urdf_description/meshes/XM,H-430_idl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 scale=0.001 0.001 0.001
- link Jaw_v4_1: geometry collision mesh filename=package://animatronics_urdf_description/meshes/Jaw_v4_1.stl scale=0.001 0.001 0.001; visual mesh filename=package://animatronics_urdf_description/meshes/Jaw_v4_1.stl scale=0.001 0.001 0.001
- link base_link: mass 1.1625557488229186 -> 5.3000587264342816; geometry collision mesh filename=package://animatronics_urdf_description/meshes/base_link.stl scale=0.001 0.001 0.001; visual mesh filename=package://animatronics_urdf_description/meshes/base_link.stl scale=0.001 0.001 0.001
Joints:
- removed joint Revolute_10
- removed joint Revolute_11
- removed joint Revolute_14
- removed joint Revolute_15
- removed joint Revolute_18
- removed joint Revolute_19
- removed joint Revolute_22
- removed joint Revolute_23
- removed joint Revolute_3
- removed joint Revolute_36
- removed joint Revolute_37
- removed joint Revolute_4
- removed joint Revolute_40
- removed joint Revolute_42
- removed joint Revolute_44
- removed joint Revolute_46
- removed joint Revolute_47
- removed joint Revolute_50
- removed joint Rigid_1
- removed joint Rigid_12
- removed joint Rigid_13
- removed joint Rigid_16
- removed joint Rigid_17
- removed joint Rigid_2
- removed joint Rigid_20
- removed joint Rigid_21
- removed joint Rigid_24
- removed joint Rigid_25
- removed joint Rigid_26
- removed joint Rigid_27
- removed joint Rigid_28
- removed joint Rigid_29
- removed joint Rigid_30
- removed joint Rigid_31
- removed joint Rigid_32
- removed joint Rigid_33
- removed joint Rigid_35
- removed joint Rigid_38
- removed joint Rigid_39
- removed joint Rigid_41
- removed joint Rigid_43
- removed joint Rigid_45
- removed joint Rigid_48
- removed joint Rigid_49
- removed joint Rigid_5
- removed joint Rigid_51
- removed joint Rigid_6
- removed joint Rigid_7
- removed joint Rigid_8
- removed joint Rigid_9
- removed joint imu_link 1_joint
- removed joint imu_link 2_joint
- removed joint imu_link 3_joint
- added joint Revolute 10: type continuous, parent 51202_v2_1, child Leg_Rotator_v10_1, origin xyz=0.0 0.012 0.0 rpy=0 0 0, axis 0.0 1.0 0.0
- added joint Revolute 12: type continuous, parent XM,H,D-540.N101.I101_v5_1, child Leg01_v11_1, origin xyz=0.0165 0.038 -0.01675 rpy=0 0 0, axis -1.0 0.0 0.0
- added joint Revolute 13: type continuous, parent Leg01_v11_1, child XM,H,D-540.N101.I101_v5_2, origin xyz=-0.0245 -0.0135 0.084 rpy=0 0 0, axis 0.0 0.0 -1.0
- added joint Revolute 16: type continuous, parent XM,H,D-540.N101.I101_v5_3, child Leg03_v28_1, origin xyz=0.018343 -0.037257 0.0165 rpy=0 0 0, axis -0.0 0.0 -1.0
- added joint Revolute 17: type continuous, parent Leg03_v28_1, child XM,H,D-540.N101.I101_v5_4, origin xyz=-0.091926 -0.077135 0.0 rpy=0 0 0, axis -0.0 0.0 -1.0
- added joint Revolute 20: type continuous, parent 51202_v2_2, child Leg_Rotator_v10_2, origin xyz=0.0 0.012 0.0 rpy=0 0 0, axis 0.0 1.0 0.0
- added joint Revolute 22: type continuous, parent XM,H,D-540.N101.I101_v5_5, child Leg01_v11_2, origin xyz=0.0165 0.038 -0.01675 rpy=0 0 0, axis -1.0 0.0 0.0
- added joint Revolute 23: type continuous, parent Leg01_v11_2, child XM,H,D-540.N101.I101_v5_6, origin xyz=-0.0245 -0.0135 -0.084 rpy=0 0 0, axis 0.0 -0.0 1.0
- added joint Revolute 26: type continuous, parent XM,H,D-540.N101.I101_v5_7, child Leg03_v28_2, origin xyz=0.039877 -0.011594 -0.0325 rpy=0 0 0, axis 0.0 -0.0 1.0
- added joint Revolute 27: type continuous, parent Leg03_v28_2, child XM,H,D-540.N101.I101_v5_8, origin xyz=-0.098298 -0.06883 0.0 rpy=0 0 0, axis 0.0 -0.0 1.0
- added joint Revolute 37: type continuous, parent base_link, child 6900ZZNR_v2_1, origin xyz=0.11025 0.05575 0.0215 rpy=0 0 0, axis -0.0 -0.0 1.0
- added joint Revolute 42: type continuous, parent Neck_Gear_Mid_Axis_v6_1, child Neck_Gear_Top_v17_1, origin xyz=0.0 0.003 0.0 rpy=0 0 0, axis 0.0 -1.0 -0.0
- added joint Revolute 43: type continuous, parent Neck_Gear_Top_v17_1, child 2XC-430_v6_1, origin xyz=0.0 0.049094 0.019 rpy=0 0 0, axis 0.0 0.0 -1.0
- added joint Revolute 44: type continuous, parent 2XC-430_v6_1, child Head_Joint_v6_1, origin xyz=-0.019 0.024 -0.019 rpy=0 0 0, axis -1.0 -0.0 -0.0
- added joint Rigid 11: type fixed, parent Leg_Rotator_v10_1, child XM,H,D-540.N101.I101_v5_1, origin xyz=0.008 0.01175 0.01675 rpy=0 0 0
- added joint Rigid 14: type fixed, parent XM,H,D-540.N101.I101_v5_2, child Leg02_v10_1, origin xyz=0.018343 -0.037257 -0.0165 rpy=0 0 0
- added joint Rigid 15: type fixed, parent Leg02_v10_1, child XM,H,D-540.N101.I101_v5_3, origin xyz=0.115374 -0.053079 0.0 rpy=0 0 0
- added joint Rigid 18: type fixed, parent XM,H,D-540.N101.I101_v5_4, child Leg04_v11_1, origin xyz=0.037258 -0.018343 -0.0165 rpy=0 0 0
- added joint Rigid 19: type fixed, parent Leg04_v11_1, child Leg_Cover_v3_1, origin xyz=0.015707 -0.066635 -0.021716 rpy=0 0 0
- added joint Rigid 21: type fixed, parent Leg_Rotator_v10_2, child XM,H,D-540.N101.I101_v5_5, origin xyz=0.008 0.01175 0.01675 rpy=0 0 0
- added joint Rigid 24: type fixed, parent XM,H,D-540.N101.I101_v5_6, child Leg02_v10_2, origin xyz=0.018343 -0.037257 0.0325 rpy=0 0 0
- added joint Rigid 25: type fixed, parent Leg02_v10_2, child XM,H,D-540.N101.I101_v5_7, origin xyz=0.09384 -0.078742 0.0 rpy=0 0 0
- added joint Rigid 28: type fixed, parent XM,H,D-540.N101.I101_v5_8, child Leg04_v11_2, origin xyz=0.035516 -0.02152 0.0165 rpy=0 0 0
- added joint Rigid 29: type fixed, parent Leg04_v11_2, child Leg_Cover_v3_2, origin xyz=0.00984 -0.06775 0.021716 rpy=0 0 0
- added joint Rigid 30: type fixed, parent base_link, child Tail_Base_v3_1, origin xyz=-0.13 -0.026 -0.035 rpy=0 0 0
- added joint Rigid 31: type fixed, parent base_link, child XM,H-430_idler_v3_1, origin xyz=0.117 0.00325 -0.0215 rpy=0 0 0
- added joint Rigid 32: type fixed, parent XM,H-430_idler_v3_1, child Neck_Gear_v10_1, origin xyz=-0.008 0.011 0.036 rpy=0 0 0
- added joint Rigid 33: type fixed, parent base_link, child Neck_Bar_v1_1, origin xyz=0.117466 0.05875 -0.0315 rpy=0 0 0
- added joint Rigid 34: type fixed, parent base_link, child Neck_Bar_v1_2, origin xyz=0.11725 0.05275 0.0315 rpy=0 0 0
- added joint Rigid 36: type fixed, parent Neck_JointH_v28_1, child 6900ZZNR_v2_2, origin xyz=0.0 0.0 -0.031 rpy=0 0 0
- added joint Rigid 38: type fixed, parent Neck_JointH_v28_1, child XL-430_new_v5_1, origin xyz=0.017 0.012522 -0.026599 rpy=0 0 0
- added joint Rigid 39: type fixed, parent XL-430_new_v5_1, child Neck_Gear_Mid_v13_1, origin xyz=0.002 0.032 0.011 rpy=0 0 0
- added joint Rigid 40: type fixed, parent XL-430_new_v5_1, child NeckMidGearHolder_v1_1, origin xyz=-0.011 0.028 0.02525 rpy=0 0 0
- added joint Rigid 41: type fixed, parent NeckMidGearHolder_v1_1, child Neck_Gear_Mid_Axis_v6_1, origin xyz=-0.006 0.01825 -0.01435 rpy=0 0 0
- added joint Rigid 45: type fixed, parent Head_Joint_v6_1, child Head_MainPlate_v4_1, origin xyz=0.0435 -0.014 -0.0285 rpy=0 0 0
- added joint Rigid 46: type fixed, parent Head_MainPlate_v4_1, child XL-430_new_v5_2, origin xyz=-0.001 -0.0095 0.0455 rpy=0 0 0
- added joint Rigid 47: type fixed, parent XL-430_new_v5_2, child Jaw_v4_1, origin xyz=0.032 -0.011 -0.036 rpy=0 0 0
- added joint Rigid 48: type fixed, parent 6900ZZNR_v2_1, child Neck_JointH_v28_1, origin xyz=0.0 0.0 -0.006 rpy=0 0 0
- added joint Rigid 6: type fixed, parent base_link, child 51202_v2_1, origin xyz=-0.099 -0.011 0.0705 rpy=0 0 0
- added joint Rigid 7: type fixed, parent base_link, child 51202_v2_2, origin xyz=-0.099 -0.011 -0.0705 rpy=0 0 0
- added joint Rigid 8: type fixed, parent base_link, child 51202_v2_3, origin xyz=-0.033 -0.011 -0.0705 rpy=0 0 0
- added joint Rigid 9: type fixed, parent base_link, child 51202_v2_4, origin xyz=-0.033 -0.011 0.0705 rpy=0 0 0
