Commit message: update robot urdf and meshes

File: animatronics_urdf_description/urdf/animatronics_urdf.xacro (robot description, xacro)
@@ -1,11 +1,11 @@
 <?xml version="1.0" ?>
-<robot name="animatronics_urdf" xmlns:xacro="http://www.ros.org/wiki/xacro">
-<xacro:include filename="$(find animatronics_urdf_description)/urdf/materials.xacro" />
-<xacro:include filename="$(find animatronics_urdf_description)/urdf/animatronics_urdf.trans" />
+<robot name="urdf" xmlns:xacro="http://www.ros.org/wiki/xacro">
+<xacro:include filename="materials.xacro" />
+<xacro:include filename="animatronics_urdf.trans" />
 <link name="base_link">
   <inertial>
-    <origin xyz="-0.03618586841730057 0.02115360522354074 0.02340251306024288" rpy="0 0 0"/>
-    <mass value="1.1625557488229186"/>
-    <inertia ixx="0.000938" iyy="0.002962" izz="0.003287" ixy="2e-06" iyz="2.7e-05" ixz="1e-06"/>
+    <origin xyz="-0.02916812257968845 -0.005246630378209138 -0.0008670637809628526" rpy="0 0 0"/>
+    <mass value="5.3000587264342816"/>
+    <inertia ixx="0.012164" iyy="0.040123" izz="0.033016" ixy="-0.002697" iyz="-0.000166" ixz="-0.000457"/>
   </inertial>
   <visual>
@@ -14,1291 +14,1076 @@
       <mesh filename="package://animatronics_urdf_description/meshes/base_link.stl" scale="0.001 0.001 0.001"/>
     </geometry>
+    <material name="steel_satin"/>
+  </visual>
+  <collision>
+    <origin xyz="0 0 0" rpy="0 0 0"/>
+    <geometry>
+      <mesh filename="package://animatronics_urdf_description/meshes/base_link.stl" scale="0.001 0.001 0.001"/>
+    </geometry>
+  </collision>
+</link>
+<link name="51202_v2_1">
+  <inertial>
+    <origin xyz="-2.674484661513432e-10 0.005999999999999998 9.590508942558529e-12" rpy="0 0 0"/>
+    <mass value="0.05505680395324213"/>
+    <inertia ixx="5e-06" iyy="8e-06" izz="5e-06" ixy="0.0" iyz="0.0" ixz="0.0"/>
+  </inertial>
+  <visual>
+    <origin xyz="0.099 0.011 -0.0705" rpy="0 0 0"/>
+    <geometry>
+      <mesh filename="package://animatronics_urdf_description/meshes/51202_v2_1.stl" scale="0.001 0.001 0.001"/>
+    </geometry>
+    <material name="steel_satin"/>
+  </visual>
+  <collision>
+    <origin xyz="0.099 0.011 -0.0705" rpy="0 0 0"/>
+    <geometry>
+      <mesh filename="package://animatronics_urdf_description/meshes/51202_v2_1.stl" scale="0.001 0.001 0.001"/>
+    </geometry>
+  </collision>
+</link>
+<link name="51202_v2_2">
+  <inertial>
+    <origin xyz="-2.764975609581555e-10 0.005999999999999998 -1.5566548050571782e-11" rpy="0 0 0"/>
+    <mass value="0.05505680395324213"/>
+    <inertia ixx="5e-06" iyy="8e-06" izz="5e-06" ixy="-0.0" iyz="0.0" ixz="-0.0"/>
+  </inertial>
+  <visual>
+    <origin xyz="0.099 0.011 0.0705" rpy="0 0 0"/>
+    <geometry>
+      <mesh filename="package://animatronics_urdf_description/meshes/51202_v2_2.stl" scale="0.001 0.001 0.001"/>
+    </geometry>
+    <material name="steel_satin"/>
+  </visual>
+  <collision>
+    <origin xyz="0.099 0.011 0.0705" rpy="0 0 0"/>
+    <geometry>
+      <mesh filename="package://animatronics_urdf_description/meshes/51202_v2_2.stl" scale="0.001 0.001 0.001"/>
+    </geometry>
+  </collision>
+</link>
+<link name="51202_v2_3">
+  <inertial>
+    <origin xyz="-2.8593932083209594e-10 0.005999999999999998 2.916361596660977e-12" rpy="0 0 0"/>
+    <mass value="0.05505680395324213"/>
+    <inertia ixx="5e-06" iyy="8e-06" izz="5e-06" ixy="0.0" iyz="0.0" ixz="0.0"/>
+  </inertial>
+  <visual>
+    <origin xyz="0.033 0.011 0.0705" rpy="0 0 0"/>
+    <geometry>
+      <mesh filename="package://animatronics_urdf_description/meshes/51202_v2_3.stl" scale="0.001 0.001 0.001"/>
+    </geometry>
+    <material name="steel_satin"/>
+  </visual>
+  <collision>
+    <origin xyz="0.033 0.011 0.0705" rpy="0 0 0"/>
+    <geometry>
+      <mesh filename="package://animatronics_urdf_description/meshes/51202_v2_3.stl" scale="0.001 0.001 0.001"/>
+    </geometry>
+  </collision>
+</link>
+<link name="51202_v2_4">
+  <inertial>
+    <origin xyz="-2.7689021214749587e-10 0.005999999999999998 -1.7363888105137448e-11" rpy="0 0 0"/>
+    <mass value="0.05505680395324213"/>
+    <inertia ixx="5e-06" iyy="8e-06" izz="5e-06" ixy="0.0" iyz="0.0" ixz="-0.0"/>
+  </inertial>
+  <visual>
+    <origin xyz="0.033 0.011 -0.0705" rpy="0 0 0"/>
+    <geometry>
+      <mesh filename="package://animatronics_urdf_description/meshes/51202_v2_4.stl" scale="0.001 0.001 0.001"/>
+    </geometry>
+    <material name="steel_satin"/>
+  </visual>
+  <collision>
+    <origin xyz="0.033 0.011 -0.0705" rpy="0 0 0"/>
+    <geometry>
+      <mesh filename="package://animatronics_urdf_description/meshes/51202_v2_4.stl" scale="0.001 0.001 0.001"/>
+    </geometry>
+  </collision>
+</link>
+<link name="Leg_Rotator_v10_1">
+  <inertial>
+    <origin xyz="0.002273583191601425 0.006491201609502772 9.179384126423162e-08" rpy="0 0 0"/>
+    <mass value="0.17090794364421608"/>
+    <inertia ixx="4.9e-05" iyy="7e-05" izz="4.4e-05" ixy="2e-06" iyz="0.0" ixz="-0.0"/>
+  </inertial>
+  <visual>
+    <origin xyz="0.099 -0.001 -0.0705" rpy="0 0 0"/>
+    <geometry>
+      <mesh filename="package://animatronics_urdf_description/meshes/Leg_Rotator_v10_1.stl" scale="0.001 0.001 0.001"/>
+    </geometry>
+    <material name="steel_satin"/>
+  </visual>
+  <collision>
+    <origin xyz="0.099 -0.001 -0.0705" rpy="0 0 0"/>
+    <geometry>
+      <mesh filename="package://animatronics_urdf_description/meshes/Leg_Rotator_v10_1.stl" scale="0.001 0.001 0.001"/>
+    </geometry>
+  </collision>
+</link>
+<link name="XM,H,D-540.N101.I101_v5_1">
+  <inertial>
+    <origin xyz="-0.007318332020298274 0.022971414590661272 -0.01674999999044581" rpy="0 0 0"/>
+    <mass value="0.6640277986148612"/>
+    <inertia ixx="0.000249" iyy="0.000169" izz="0.000301" ixy="-1e-06" iyz="0.0" ixz="-0.0"/>
+  </inertial>
+  <visual>
+    <origin xyz="0.091 -0.01275 -0.08725" rpy="0 0 0"/>
+    <geometry>
+      <mesh filename="package://animatronics_urdf_description/meshes/XM,H,D-540.N101.I101_v5_1.stl" scale="0.001 0.001 0.001"/>
+    </geometry>
+    <material name="coating_black_oxide"/>
+  </visual>
+  <collision>
+    <origin xyz="0.091 -0.01275 -0.08725" rpy="0 0 0"/>
+    <geometry>
+      <mesh filename="package://animatronics_urdf_description/meshes/XM,H,D-540.N101.I101_v5_1.stl" scale="0.001 0.001 0.001"/>
+    </geometry>
+  </collision>
+</link>
+<link name="Leg01_v11_1">
+  <inertial>
+    <origin xyz="-0.02449977648783827 0.003928976257230828 0.04188393608676076" rpy="0 0 0"/>
+    <mass value="0.244537289734516"/>
+    <inertia ixx="0.000195" iyy="0.000256" izz="0.000113" ixy="0.0" iyz="-1.6e-05" ixz="0.0"/>
+  </inertial>
+  <visual>
+    <origin xyz="0.0745 -0.05075 -0.0705" rpy="0 0 0"/>
+    <geometry>
+      <mesh filename="package://animatronics_urdf_description/meshes/Leg01_v11_1.stl" scale="0.001 0.001 0.001"/>
+    </geometry>
+    <material name="steel_satin"/>
+  </visual>
+  <collision>
+    <origin xyz="0.0745 -0.05075 -0.0705" rpy="0 0 0"/>
+    <geometry>
+      <mesh filename="package://animatronics_urdf_description/meshes/Leg01_v11_1.stl" scale="0.001 0.001 0.001"/>
+    </geometry>
+  </collision>
+</link>
+<link name="XM,H,D-540.N101.I101_v5_2">
+  <inertial>
+    <origin xyz="0.011512563950167629 -0.009660188724108575 -0.023818331012862903" rpy="0 0 0"/>
+    <mass value="0.6640277986148612"/>
+    <inertia ixx="0.000224" iyy="0.000247" izz="0.000249" ixy="6.5e-05" iyz="-1e-06" ixz="1e-06"/>
+  </inertial>
+  <visual>
+    <origin xyz="0.099 -0.03725 -0.1545" rpy="0 0 0"/>
+    <geometry>
+      <mesh filename="package://animatronics_urdf_description/meshes/XM,H,D-540.N101.I101_v5_2.stl" scale="0.001 0.001 0.001"/>
+    </geometry>
+    <material name="coating_black_oxide"/>
+  </visual>
+  <collision>
+    <origin xyz="0.099 -0.03725 -0.1545" rpy="0 0 0"/>
+    <geometry>
+      <mesh filename="package://animatronics_urdf_description/meshes/XM,H,D-540.N101.I101_v5_2.stl" scale="0.001 0.001 0.001"/>
+    </geometry>
+  </collision>
+</link>
+<link name="Leg02_v10_1">
+  <inertial>
+    <origin xyz="0.05768691058893847 -0.026539670493288297 -0.007999999260265594" rpy="0 0 0"/>
+    <mass value="0.7208590729525296"/>
+    <inertia ixx="0.000716" iyy="0.000873" izz="0.001271" ixy="0.000444" iyz="0.0" ixz="0.0"/>
+  </inertial>
+  <visual>
+    <origin xyz="0.080657 7e-06 -0.138" rpy="0 0 0"/>
+    <geometry>
+      <mesh filename="package://animatronics_urdf_description/meshes/Leg02_v10_1.stl" scale="0.001 0.001 0.001"/>
+    </geometry>
+    <material name="steel_satin"/>
+  </visual>
+  <collision>
+    <origin xyz="0.080657 7e-06 -0.138" rpy="0 0 0"/>
+    <geometry>
+      <mesh filename="package://animatronics_urdf_description/meshes/Leg02_v10_1.stl" scale="0.001 0.001 0.001"/>
+    </geometry>
+  </collision>
+</link>
+<link name="XM,H,D-540.N101.I101_v5_3">
+  <inertial>
+    <origin xyz="0.0068302572277092535 -0.027597152262468012 -0.007318331012862972" rpy="0 0 0"/>
+    <mass value="0.6640277986148612"/>
+    <inertia ixx="0.000224" iyy="0.000247" izz="0.000249" ixy="6.5e-05" iyz="1e-06" ixz="-1e-06"/>
+  </inertial>
+  <visual>
+    <origin xyz="-0.034717 0.053086 -0.138" rpy="0 0 0"/>
+    <geometry>
+      <mesh filename="package://animatronics_urdf_description/meshes/XM,H,D-540.N101.I101_v5_3.stl" scale="0.001 0.001 0.001"/>
+    </geometry>
+    <material name="coating_black_oxide"/>
+  </visual>
+  <collision>
+    <origin xyz="-0.034717 0.053086 -0.138" rpy="0 0 0"/>
+    <geometry>
+      <mesh filename="package://animatronics_urdf_description/meshes/XM,H,D-540.N101.I101_v5_3.stl" scale="0.001 0.001 0.001"/>
+    </geometry>
+  </collision>
+</link>
+<link name="Leg03_v28_1">
+  <inertial>
+    <origin xyz="-0.04600850374218349 -0.038605909178262204 -0.024469720937909306" rpy="0 0 0"/>
+    <mass value="0.0705061968864148"/>
+    <inertia ixx="6.4e-05" iyy="7.2e-05" izz="6.5e-05" ixy="-2.2e-05" iyz="0.0" ixz="0.0"/>
+  </inertial>
+  <visual>
+    <origin xyz="-0.05306 0.090343 -0.1545" rpy="0 0 0"/>
+    <geometry>
+      <mesh filename="package://animatronics_urdf_description/meshes/Leg03_v28_1.stl" scale="0.001 0.001 0.001"/>
+    </geometry>
+    <material name="plastic_translucent_glossy_white"/>
+  </visual>
+  <collision>
+    <origin xyz="-0.05306 0.090343 -0.1545" rpy="0 0 0"/>
+    <geometry>
+      <mesh filename="package://animatronics_urdf_description/meshes/Leg03_v28_1.stl" scale="0.001 0.001 0.001"/>
+    </geometry>
+  </collision>
+</link>
+<link name="XM,H,D-540.N101.I101_v5_4">
+  <inertial>
+    <origin xyz="0.009660676886473377 -0.011512418257745072 -0.023818331012863014" rpy="0 0 0"/>
+    <mass value="0.6640277986148612"/>
+    <inertia ixx="0.000247" iyy="0.000224" izz="0.000249" ixy="6.5e-05" iyz="-1e-06" ixz="1e-06"/>
+  </inertial>
+  <visual>
+    <origin xyz="0.038866 0.167478 -0.1545" rpy="0 0 0"/>
+    <geometry>
+      <mesh filename="package://animatronics_urdf_description/meshes/XM,H,D-540.N101.I101_v5_4.stl" scale="0.001 0.001 0.001"/>
+    </geometry>
+    <material name="coating_black_oxide"/>
+  </visual>
+  <collision>
+    <origin xyz="0.038866 0.167478 -0.1545" rpy="0 0 0"/>
+    <geometry>
+      <mesh filename="package://animatronics_urdf_description/meshes/XM,H,D-540.N101.I101_v5_4.stl" scale="0.001 0.001 0.001"/>
+    </geometry>
+  </collision>
+</link>
+<link name="Leg04_v11_1">
+  <inertial>
+    <origin xyz="0.018979657861121692 -0.04035064948330955 -0.008000009830100047" rpy="0 0 0"/>
+    <mass value="1.201075021531332"/>
+    <inertia ixx="0.000647" iyy="0.001024" izz="0.001001" ixy="0.000253" iyz="-0.0" ixz="-0.0"/>
+  </inertial>
+  <visual>
+    <origin xyz="0.001608 0.185821 -0.138" rpy="0 0 0"/>
+    <geometry>
+      <mesh filename="package://animatronics_urdf_description/meshes/Leg04_v11_1.stl" scale="0.001 0.001 0.001"/>
+    </geometry>
+    <material name="steel_satin"/>
+  </visual>
+  <collision>
+    <origin xyz="0.001608 0.185821 -0.138" rpy="0 0 0"/>
+    <geometry>
+      <mesh filename="package://animatronics_urdf_description/meshes/Leg04_v11_1.stl" scale="0.001 0.001 0.001"/>
+    </geometry>
+  </collision>
+</link>
+<link name="Leg_Cover_v3_1">
+  <inertial>
+    <origin xyz="0.022608679812465393 -0.0008954873889764348 0.013716000739732392" rpy="0 0 0"/>
+    <mass value="0.15624009364552216"/>
+    <inertia ixx="5.2e-05" iyy="9.1e-05" izz="4e-05" ixy="-4e-06" iyz="-0.0" ixz="-0.0"/>
+  </inertial>
+  <visual>
+    <origin xyz="-0.014099 0.252456 -0.116284" rpy="0 0 0"/>
+    <geometry>
+      <mesh filename="package://animatronics_urdf_description/meshes/Leg_Cover_v3_1.stl" scale="0.001 0.001 0.001"/>
+    </geometry>
+    <material name="steel_satin"/>
+  </visual>
+  <collision>
+    <origin xyz="-0.014099 0.252456 -0.116284" rpy="0 0 0"/>
+    <geometry>
+      <mesh filename="package://animatronics_urdf_description/meshes/Leg_Cover_v3_1.stl" scale="0.001 0.001 0.001"/>
+    </geometry>
+  </collision>
+</link>
+<link name="Leg_Rotator_v10_2">
+  <inertial>
+    <origin xyz="0.0022735831825523023 0.006491201609502772 9.176868422111628e-08" rpy="0 0 0"/>
+    <mass value="0.17090794364421608"/>
+    <inertia ixx="4.9e-05" iyy="7e-05" izz="4.4e-05" ixy="2e-06" iyz="0.0" ixz="-0.0"/>
+  </inertial>
+  <visual>
+    <origin xyz="0.099 -0.001 0.0705" rpy="0 0 0"/>
+    <geometry>
+      <mesh filename="package://animatronics_urdf_description/meshes/Leg_Rotator_v10_2.stl" scale="0.001 0.001 0.001"/>
+    </geometry>
+    <material name="steel_satin"/>
+  </visual>
+  <collision>
+    <origin xyz="0.099 -0.001 0.0705" rpy="0 0 0"/>
+    <geometry>
+      <mesh filename="package://animatronics_urdf_description/meshes/Leg_Rotator_v10_2.stl" scale="0.001 0.001 0.001"/>
+    </geometry>
+  </collision>
+</link>
+<link name="XM,H,D-540.N101.I101_v5_5">
+  <inertial>
+    <origin xyz="-0.00731833202934741 0.022971414590661272 -0.01675000001560286" rpy="0 0 0"/>
+    <mass value="0.6640277986148612"/>
+    <inertia ixx="0.000249" iyy="0.000169" izz="0.000301" ixy="-1e-06" iyz="0.0" ixz="-0.0"/>
+  </inertial>
+  <visual>
+    <origin xyz="0.091 -0.01275 0.05375" rpy="0 0 0"/>
+    <geometry>
+      <mesh filename="package://animatronics_urdf_description/meshes/XM,H,D-540.N101.I101_v5_5.stl" scale="0.001 0.001 0.001"/>
+    </geometry>
+    <material name="coating_black_oxide"/>
+  </visual>
+  <collision>
+    <origin xyz="0.091 -0.01275 0.05375" rpy="0 0 0"/>
+    <geometry>
+      <mesh filename="package://animatronics_urdf_description/meshes/XM,H,D-540.N101.I101_v5_5.stl" scale="0.001 0.001 0.001"/>
+    </geometry>
+  </collision>
+</link>
+<link name="Leg01_v11_2">
+  <inertial>
+    <origin xyz="-0.0245002244253857 0.003928976303331326 -0.04188393609273208" rpy="0 0 0"/>
+    <mass value="0.244537289734516"/>
+    <inertia ixx="0.000195" iyy="0.000256" izz="0.000113" ixy="-0.0" iyz="1.6e-05" ixz="0.0"/>
+  </inertial>
+  <visual>
+    <origin xyz="0.0745 -0.05075 0.0705" rpy="0 0 0"/>
+    <geometry>
+      <mesh filename="package://animatronics_urdf_description/meshes/Leg01_v11_2.stl" scale="0.001 0.001 0.001"/>
+    </geometry>
+    <material name="steel_satin"/>
+  </visual>
+  <collision>
+    <origin xyz="0.0745 -0.05075 0.0705" rpy="0 0 0"/>
+    <geometry>
+      <mesh filename="package://animatronics_urdf_description/meshes/Leg01_v11_2.stl" scale="0.001 0.001 0.001"/>
+    </geometry>
+  </collision>
+</link>
+<link name="XM,H,D-540.N101.I101_v5_6">
+  <inertial>
+    <origin xyz="0.011512563818134161 -0.009660188678067217 0.02381833100689157" rpy="0 0 0"/>
+    <mass value="0.6640277986148612"/>
+    <inertia ixx="0.000224" iyy="0.000247" izz="0.000249" ixy="6.5e-05" iyz="1e-06" ixz="-1e-06"/>
+  </inertial>
+  <visual>
+    <origin xyz="0.099 -0.03725 0.1545" rpy="0 0 0"/>
+    <geometry>
+      <mesh filename="package://animatronics_urdf_description/meshes/XM,H,D-540.N101.I101_v5_6.stl" scale="0.001 0.001 0.001"/>
+    </geometry>
+    <material name="coating_black_oxide"/>
+  </visual>
+  <collision>
+    <origin xyz="0.099 -0.03725 0.1545" rpy="0 0 0"/>
+    <geometry>
+      <mesh filename="package://animatronics_urdf_description/meshes/XM,H,D-540.N101.I101_v5_6.stl" scale="0.001 0.001 0.001"/>
+    </geometry>
+  </collision>
+</link>
+<link name="Leg02_v10_2">
+  <inertial>
+    <origin xyz="0.05768691045695463 -0.026539670447187826 -0.008000000745736563" rpy="0 0 0"/>
+    <mass value="0.7208590729525296"/>
+    <inertia ixx="0.000716" iyy="0.000873" izz="0.001271" ixy="0.000444" iyz="-0.0" ixz="-0.0"/>
+  </inertial>
+  <visual>
+    <origin xyz="0.080657 7e-06 0.122" rpy="0 0 0"/>
+    <geometry>
+      <mesh filename="package://animatronics_urdf_description/meshes/Leg02_v10_2.stl" scale="0.001 0.001 0.001"/>
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
File: animatronics_urdf_description/urdf/materials.xacro (robot description, xacro)
@@ -1,9 +1,9 @@
 <?xml version="1.0" ?>
-<robot name="animatronics_urdf" xmlns:xacro="http://www.ros.org/wiki/xacro" >
+<robot name="urdf" xmlns:xacro="http://www.ros.org/wiki/xacro" >
 <material name="silver_default">
   <color rgba="0.700 0.700 0.700 1.000"/>
 </material>
-<material name="plastic_glossy_white">
-  <color rgba="0.9647058823529412 0.9647058823529412 0.9529411764705882 1.0"/>
+<material name="steel_satin">
+  <color rgba="0.6274509803921569 0.6274509803921569 0.6274509803921569 1.0"/>
 </material>
 <material name="coating_black_oxide">
@@ -13,15 +13,9 @@
   <color rgba="0.9647058823529412 0.9647058823529412 0.9529411764705882 1.0"/>
 </material>
-<material name="steel_satin">
-  <color rgba="0.6274509803921569 0.6274509803921569 0.6274509803921569 1.0"/>
-</material>
-<material name="nylon_12_with_formlabs_fuse_1_3d_printer">
-  <color rgba="0.24705882352941178 0.24705882352941178 0.24705882352941178 1.0"/>
-</material>
 <material name="abs_white">
   <color rgba="0.9647058823529412 0.9647058823529412 0.9529411764705882 1.0"/>
 </material>
-<material name="opaque198193188">
-  <color rgba="0.7764705882352941 0.7568627450980392 0.7372549019607844 1.0"/>
+<material name="plastic_glossy_white">
+  <color rgba="0.9647058823529412 0.9647058823529412 0.9529411764705882 1.0"/>
 </material>
 <material name="opaque160160160">

Commit message: update robot urdf and meshes

File: animatronics_urdf_description/animatronics_urdf_description_standalone.urdf (robot description, URDF)
Before this commit: robot urdf, 43 links, 42 joints
Links:
- added link 51202_v2_5, mass 0.05505680395324213; collision mesh filename=package://animatronics_urdf_description/meshes/51202_v2_5.s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 scale=0.001 0.001 0.001; visual mesh filename=package://animatronics_urdf_description/meshes/51202_v2_5.s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 scale=0.001 0.001 0.001
- added link 51202_v2_6, mass 0.05505680395324213; collision mesh filename=package://animatronics_urdf_description/meshes/51202_v2_6.s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 scale=0.001 0.001 0.001; visual mesh filename=package://animatronics_urdf_description/meshes/51202_v2_6.s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 scale=0.001 0.001 0.001
- added link Leg_Rotator_Upper_v4_1, mass 0.07969136297131019; collision mesh filename=package://animatronics_urdf_description/meshes/Leg_Rotator_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 scale=0.001 0.001 0.001; visual mesh filename=package://animatronics_urdf_description/meshes/Leg_Rotator_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 scale=0.001 0.001 0.001
- added link Leg_Rotator_Upper_v4_2, mass 0.07969136297131019; collision mesh filename=package://animatronics_urdf_description/meshes/Leg_Rotator_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 scale=0.001 0.001 0.001; visual mesh filename=package://animatronics_urdf_description/meshes/Leg_Rotator_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 scale=0.001 0.001 0.001
- added link body_cover_v21_1, mass 2.0845144413763554; collision mesh filename=package://animatronics_urdf_description/meshes/body_cover_v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 scale=0.001 0.001 0.001; visual mesh filename=package://animatronics_urdf_description/meshes/body_cover_v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 scale=0.001 0.001 0.001
Joints:
- added joint Rigid 49: type fixed, parent XM,H,D-540.N101.I101_v5_1, child Leg_Rotator_Upper_v4_1, origin xyz=0.0 0.032 0.0 rpy=0 0 0
- added joint Rigid 50: type fixed, parent Leg_Rotator_Upper_v4_1, child 51202_v2_5, origin xyz=-0.008 0.02375 -0.01675 rpy=0 0 0
- added joint Rigid 51: type fixed, parent XM,H,D-540.N101.I101_v5_5, child Leg_Rotator_Upper_v4_2, origin xyz=0.0 0.032 0.0 rpy=0 0 0
- added joint Rigid 52: type fixed, parent Leg_Rotator_Upper_v4_2, child 51202_v2_6, origin xyz=-0.008 0.02375 -0.01675 rpy=0 0 0
- added joint Rigid 58: type fixed, parent base_link, child body_cover_v21_1, origin xyz=-0.125 0.0385 0.0 rpy=0 0 0
- joint Revolute 17: origin xyz=-0.091926 -0.077135 0.0 rpy=0 0 0 -> xyz=-0.077135 -0.091926 0.0 rpy=0 0 0
- joint Revolute 26: axis 0.0 -0.0 1.0 -> -0.0 -0.0 1.0
- joint Revolute 27: origin xyz=-0.098298 -0.06883 0.0 rpy=0 0 0 -> xyz=-0.077135 -0.091926 0.0 rpy=0 0 0
- joint Revolute 42: axis 0.0 -1.0 -0.0 -> -0.422618 -0.906308 -0.0; origin xyz=0.0 0.003 0.0 rpy=0 0 0 -> xyz=0.001268 0.002719 0.0 rpy=0 0 0
- joint Revolute 43: origin xyz=0.0 0.049094 0.019 rpy=0 0 0 -> xyz=0.020748 0.044494 0.019 rpy=0 0 0
- joint Rigid 18: origin xyz=0.037258 -0.018343 -0.0165 rpy=0 0 0 -> xyz=0.035517 -0.02152 -0.0165 rpy=0 0 0
- joint Rigid 19: origin xyz=0.015707 -0.066635 -0.021716 rpy=0 0 0 -> xyz=0.00984 -0.06775 -0.021716 rpy=0 0 0
- joint Rigid 28: origin xyz=0.035516 -0.02152 0.0165 rpy=0 0 0 -> xyz=0.035517 -0.02152 0.0165 rpy=0 0 0
- joint Rigid 38: origin xyz=0.017 0.012522 -0.026599 rpy=0 0 0 -> xyz=0.020699 0.004164 -0.026599 rpy=0 0 0
- joint Rigid 39: origin xyz=0.002 0.032 0.011 rpy=0 0 0 -> xyz=0.015337 0.028157 0.011 rpy=0 0 0
- joint Rigid 40: origin xyz=-0.011 0.028 0.02525 rpy=0 0 0 -> xyz=0.001864 0.030026 0.02525 rpy=0 0 0
- joint Rigid 41: origin xyz=-0.006 0.01825 -0.01435 rpy=0 0 0 -> xyz=0.002275 0.019075 -0.01435 rpy=0 0 0
