Commit message: update robot urdf and meshes

File: animatronics_urdf_description/urdf/animatronics_urdf.xacro (robot description, xacro)
@@ -165,5 +165,5 @@
 <link name="XM,H,D-540.N101.I101_v5_2">
   <inertial>
-    <origin xyz="0.011512563950167629 -0.009660188724108575 -0.023818331012862903" rpy="0 0 0"/>
+    <origin xyz="0.011512563950167629 -0.00966018872410861 -0.023818331012862903" rpy="0 0 0"/>
     <mass value="0.6640277986148612"/>
     <inertia ixx="0.000224" iyy="0.000247" izz="0.000249" ixy="6.5e-05" iyz="-1e-06" ixz="1e-06"/>
@@ -185,5 +185,5 @@
 <link name="Leg02_v10_1">
   <inertial>
-    <origin xyz="0.05768691058893847 -0.026539670493288297 -0.007999999260265594" rpy="0 0 0"/>
+    <origin xyz="0.057686910588938496 -0.02653967049328852 -0.007999999260265594" rpy="0 0 0"/>
     <mass value="0.7208590729525296"/>
     <inertia ixx="0.000716" iyy="0.000873" izz="0.001271" ixy="0.000444" iyz="0.0" ixz="0.0"/>
@@ -205,5 +205,5 @@
 <link name="XM,H,D-540.N101.I101_v5_3">
   <inertial>
-    <origin xyz="0.0068302572277092535 -0.027597152262468012 -0.007318331012862972" rpy="0 0 0"/>
+    <origin xyz="0.006830257227709316 -0.02759715226246829 -0.007318331012862944" rpy="0 0 0"/>
     <mass value="0.6640277986148612"/>
     <inertia ixx="0.000224" iyy="0.000247" izz="0.000249" ixy="6.5e-05" iyz="1e-06" ixz="-1e-06"/>
@@ -225,7 +225,7 @@
 <link name="Leg03_v28_1">
   <inertial>
-    <origin xyz="-0.04600850374218349 -0.038605909178262204 -0.024469720937909306" rpy="0 0 0"/>
+    <origin xyz="-0.03860574729601735 -0.046008665695374346 -0.024469720937909195" rpy="0 0 0"/>
     <mass value="0.0705061968864148"/>
-    <inertia ixx="6.4e-05" iyy="7.2e-05" izz="6.5e-05" ixy="-2.2e-05" iyz="0.0" ixz="0.0"/>
+    <inertia ixx="7.2e-05" iyy="6.4e-05" izz="6.5e-05" ixy="-2.2e-05" iyz="0.0" ixz="0.0"/>
   </inertial>
   <visual>
@@ -245,10 +245,10 @@
 <link name="XM,H,D-540.N101.I101_v5_4">
   <inertial>
-    <origin xyz="0.009660676886473377 -0.011512418257745072 -0.023818331012863014" rpy="0 0 0"/>
+    <origin xyz="0.008620350868605839 -0.01231037038971286 -0.023818331012862903" rpy="0 0 0"/>
     <mass value="0.6640277986148612"/>
-    <inertia ixx="0.000247" iyy="0.000224" izz="0.000249" ixy="6.5e-05" iyz="-1e-06" ixz="1e-06"/>
-  </inertial>
-  <visual>
-    <origin xyz="0.038866 0.167478 -0.1545" rpy="0 0 0"/>
+    <inertia ixx="0.000258" iyy="0.000213" izz="0.000249" ixy="6.2e-05" iyz="-1e-06" ixz="1e-06"/>
+  </inertial>
+  <visual>
+    <origin xyz="0.024075 0.182269 -0.1545" rpy="0 0 0"/>
     <geometry>
       <mesh filename="package://animatronics_urdf_description/meshes/XM,H,D-540.N101.I101_v5_4.stl" scale="0.001 0.001 0.001"/>
@@ -257,5 +257,5 @@
   </visual>
   <collision>
-    <origin xyz="0.038866 0.167478 -0.1545" rpy="0 0 0"/>
+    <origin xyz="0.024075 0.182269 -0.1545" rpy="0 0 0"/>
     <geometry>
       <mesh filename="package://animatronics_urdf_description/meshes/XM,H,D-540.N101.I101_v5_4.stl" scale="0.001 0.001 0.001"/>
@@ -265,10 +265,10 @@
 <link name="Leg04_v11_1">
   <inertial>
-    <origin xyz="0.018979657861121692 -0.04035064948330955 -0.008000009830100047" rpy="0 0 0"/>
+    <origin xyz="0.015390977117457464 -0.04185151415784971 -0.008000009830099908" rpy="0 0 0"/>
     <mass value="1.201075021531332"/>
-    <inertia ixx="0.000647" iyy="0.001024" izz="0.001001" ixy="0.000253" iyz="-0.0" ixz="-0.0"/>
-  </inertial>
-  <visual>
-    <origin xyz="0.001608 0.185821 -0.138" rpy="0 0 0"/>
+    <inertia ixx="0.000693" iyy="0.000977" izz="0.001001" ixy="0.000282" iyz="-0.0" ixz="-0.0"/>
+  </inertial>
+  <visual>
+    <origin xyz="-0.011442 0.203789 -0.138" rpy="0 0 0"/>
     <geometry>
       <mesh filename="package://animatronics_urdf_description/meshes/Leg04_v11_1.stl" scale="0.001 0.001 0.001"/>
@@ -277,5 +277,5 @@
   </visual>
   <collision>
-    <origin xyz="0.001608 0.185821 -0.138" rpy="0 0 0"/>
+    <origin xyz="-0.011442 0.203789 -0.138" rpy="0 0 0"/>
     <geometry>
       <mesh filename="package://animatronics_urdf_description/meshes/Leg04_v11_1.stl" scale="0.001 0.001 0.001"/>
@@ -285,10 +285,10 @@
 <link name="Leg_Cover_v3_1">
   <inertial>
-    <origin xyz="0.022608679812465393 -0.0008954873889764348 0.013716000739732392" rpy="0 0 0"/>
+    <origin xyz="0.02244454070714232 -0.002863169929422704 0.013716000739732531" rpy="0 0 0"/>
     <mass value="0.15624009364552216"/>
-    <inertia ixx="5.2e-05" iyy="9.1e-05" izz="4e-05" ixy="-4e-06" iyz="-0.0" ixz="-0.0"/>
-  </inertial>
-  <visual>
-    <origin xyz="-0.014099 0.252456 -0.116284" rpy="0 0 0"/>
+    <inertia ixx="5.2e-05" iyy="9.1e-05" izz="4e-05" ixy="-0.0" iyz="-0.0" ixz="-0.0"/>
+  </inertial>
+  <visual>
+    <origin xyz="-0.021282 0.271539 -0.116284" rpy="0 0 0"/>
     <geometry>
       <mesh filename="package://animatronics_urdf_description/meshes/Leg_Cover_v3_1.stl" scale="0.001 0.001 0.001"/>
@@ -297,5 +297,5 @@
   </visual>
   <collision>
-    <origin xyz="-0.014099 0.252456 -0.116284" rpy="0 0 0"/>
+    <origin xyz="-0.021282 0.271539 -0.116284" rpy="0 0 0"/>
     <geometry>
       <mesh filename="package://animatronics_urdf_description/meshes/Leg_Cover_v3_1.stl" scale="0.001 0.001 0.001"/>
@@ -365,5 +365,5 @@
 <link name="XM,H,D-540.N101.I101_v5_6">
   <inertial>
-    <origin xyz="0.011512563818134161 -0.009660188678067217 0.02381833100689157" rpy="0 0 0"/>
+    <origin xyz="0.011512563818134189 -0.009660188678067227 0.02381833100689157" rpy="0 0 0"/>
     <mass value="0.6640277986148612"/>
     <inertia ixx="0.000224" iyy="0.000247" izz="0.000249" ixy="6.5e-05" iyz="1e-06" ixz="-1e-06"/>
@@ -385,5 +385,5 @@
 <link name="Leg02_v10_2">
   <inertial>
-    <origin xyz="0.05768691045695463 -0.026539670447187826 -0.008000000745736563" rpy="0 0 0"/>
+    <origin xyz="0.05768691045695482 -0.026539670447187833 -0.008000000745736618" rpy="0 0 0"/>
     <mass value="0.7208590729525296"/>
     <inertia ixx="0.000716" iyy="0.000873" izz="0.001271" ixy="0.000444" iyz="-0.0" ixz="-0.0"/>
@@ -405,5 +405,5 @@
 <link name="XM,H,D-540.N101.I101_v5_7">
   <inertial>
-    <origin xyz="0.02836425709577517 -0.0019341522163084657 -0.008681668993108432" rpy="0 0 0"/>
+    <origin xyz="0.02836425709577542 -0.0019341522163085073 -0.008681668993108432" rpy="0 0 0"/>
     <mass value="0.6640277986148612"/>
     <inertia ixx="0.000224" iyy="0.000247" izz="0.000249" ixy="6.5e-05" iyz="-1e-06" ixz="1e-06"/>
@@ -425,7 +425,7 @@
 <link name="Leg03_v28_2">
   <inertial>
-    <origin xyz="-0.049198125296219974 -0.0344491135239421 0.024530277576619824" rpy="0 0 0"/>
+    <origin xyz="-0.03860574742800091 -0.046008665649273806 0.024530277576619797" rpy="0 0 0"/>
     <mass value="0.0705061968864148"/>
-    <inertia ixx="6e-05" iyy="7.5e-05" izz="6.5e-05" ixy="-2.1e-05" iyz="0.0" ixz="0.0"/>
+    <inertia ixx="7.2e-05" iyy="6.4e-05" izz="6.5e-05" ixy="-2.2e-05" iyz="0.0" ixz="0.0"/>
   </inertial>
   <visual>
@@ -445,10 +445,10 @@
 <link name="XM,H,D-540.N101.I101_v5_8">
   <inertial>
-    <origin xyz="0.00861961858427858 -0.012310209531500138 0.023818331006891513" rpy="0 0 0"/>
+    <origin xyz="0.00862035073655892 -0.012310370343656785 0.023818331006891513" rpy="0 0 0"/>
     <mass value="0.6640277986148612"/>
     <inertia ixx="0.000258" iyy="0.000213" izz="0.000249" ixy="6.2e-05" iyz="1e-06" ixz="-1e-06"/>
   </inertial>
   <visual>
-    <origin xyz="0.045238 0.159173 0.1545" rpy="0 0 0"/>
+    <origin xyz="0.024075 0.182269 0.1545" rpy="0 0 0"/>
     <geometry>
       <mesh filename="package://animatronics_urdf_description/meshes/XM,H,D-540.N101.I101_v5_8.stl" scale="0.001 0.001 0.001"/>
@@ -457,5 +457,5 @@
   </visual>
   <collision>
-    <origin xyz="0.045238 0.159173 0.1545" rpy="0 0 0"/>
+    <origin xyz="0.024075 0.182269 0.1545" rpy="0 0 0"/>
     <geometry>
       <mesh filename="package://animatronics_urdf_description/meshes/XM,H,D-540.N101.I101_v5_8.stl" scale="0.001 0.001 0.001"/>
@@ -465,10 +465,10 @@
 <link name="Leg04_v11_2">
   <inertial>
-    <origin xyz="0.015391244833193509 -0.04185135329959272 0.007999988684428999" rpy="0 0 0"/>
+    <origin xyz="0.015390976985473911 -0.041851514111749366 0.007999988684428999" rpy="0 0 0"/>
     <mass value="1.201075021531332"/>
     <inertia ixx="0.000693" iyy="0.000977" izz="0.001001" ixy="0.000282" iyz="-0.0" ixz="-0.0"/>
   </inertial>
   <visual>
-    <origin xyz="0.009722 0.180693 0.138" rpy="0 0 0"/>
+    <origin xyz="-0.011442 0.203789 0.138" rpy="0 0 0"/>
     <geometry>
       <mesh filename="package://animatronics_urdf_description/meshes/Leg04_v11_2.stl" scale="0.001 0.001 0.001"/>
@@ -477,5 +477,5 @@
   </visual>
   <collision>
-    <origin xyz="0.009722 0.180693 0.138" rpy="0 0 0"/>
+    <origin xyz="-0.011442 0.203789 0.138" rpy="0 0 0"/>
     <geometry>
       <mesh filename="package://animatronics_urdf_description/meshes/Leg04_v11_2.stl" scale="0.001 0.001 0.001"/>
@@ -485,10 +485,10 @@
 <link name="Leg_Cover_v3_2">
   <inertial>
-    <origin xyz="0.02244480842287839 -0.002863009071165573 -0.013716000745738616" rpy="0 0 0"/>
+    <origin xyz="0.022444540575158847 -0.0028631698833221364 -0.013716000745738616" rpy="0 0 0"/>
     <mass value="0.15624009364552216"/>
     <inertia ixx="5.2e-05" iyy="9.1e-05" izz="4e-05" ixy="-0.0" iyz="-0.0" ixz="-0.0"/>
   </inertial>
   <visual>
-    <origin xyz="-0.000118 0.248443 0.116284" rpy="0 0 0"/>
+    <origin xyz="-0.021282 0.271539 0.116284" rpy="0 0 0"/>
     <geometry>
       <mesh filename="package://animatronics_urdf_description/meshes/Leg_Cover_v3_2.stl" scale="0.001 0.001 0.001"/>
@@ -497,5 +497,5 @@
   </visual>
   <collision>
-    <origin xyz="-0.000118 0.248443 0.116284" rpy="0 0 0"/>
+    <origin xyz="-0.021282 0.271539 0.116284" rpy="0 0 0"/>
     <geometry>
       <mesh filename="package://animatronics_urdf_description/meshes/Leg_Cover_v3_2.stl" scale="0.001 0.001 0.001"/>
@@ -605,7 +605,7 @@
 <link name="6900ZZNR_v2_2">
   <inertial>
-    <origin xyz="6.566552857023567e-13 5.745404152435185e-15 -0.0030000000173622914" rpy="0 0 0"/>
+    <origin xyz="6.693118281830834e-13 6.320638457069094e-14 -0.003000000017362319" rpy="0 0 0"/>
     <mass value="0.014205025342471455"/>
-    <inertia ixx="1e-06" iyy="1e-06" izz="1e-06" ixy="0.0" iyz="-0.0" ixz="-0.0"/>
+    <inertia ixx="1e-06" iyy="1e-06" izz="1e-06" ixy="-0.0" iyz="-0.0" ixz="-0.0"/>
   </inertial>
   <visual>
@@ -625,7 +625,7 @@
 <link name="6900ZZNR_v2_1">
   <inertial>
-    <origin xyz="6.082079284652764e-13 4.163336342344337e-16 -0.0030000000173622567" rpy="0 0 0"/>
+    <origin xyz="6.209616154606579e-13 5.796058077933708e-14 -0.0030000000173622567" rpy="0 0 0"/>
     <mass value="0.014205025342471455"/>
-    <inertia ixx="1e-06" iyy="1e-06" izz="1e-06" ixy="0.0" iyz="-0.0" ixz="-0.0"/>
+    <inertia ixx="1e-06" iyy="1e-06" izz="1e-06" ixy="-0.0" iyz="-0.0" ixz="-0.0"/>
   </inertial>
   <visual>
@@ -645,10 +645,10 @@
 <link name="XL-430_new_v5_1">
   <inertial>
-    <origin xyz="-0.016334115662739873 0.020332402663781793 0.011008281617759614" rpy="0 0 0"/>
+    <origin xyz="-0.006210633295508319 0.025330786091814946 0.011008281617777189" rpy="0 0 0"/>
     <mass value="0.33677880262575866"/>
-    <inertia ixx="8.2e-05" iyy="5.5e-05" izz="9.4e-05" ixy="-0.0" iyz="-0.0" ixz="-0.0"/>
-  </inertial>
-  <visual>
-    <origin xyz="-0.12725 -0.068272 0.011099" rpy="0 0 0"/>
+    <inertia ixx="7.7e-05" iyy="6e-05" izz="9.4e-05" ixy="-1.1e-05" iyz="-0.0" ixz="-0.0"/>
+  </inertial>
+  <visual>
+    <origin xyz="-0.130949 -0.059914 0.011099" rpy="0 0 0"/>
     <geometry>
       <mesh filename="package://animatronics_urdf_description/meshes/XL-430_new_v5_1.stl" scale="0.001 0.001 0.001"/>
@@ -657,5 +657,5 @@
   </visual>
   <collision>
-    <origin xyz="-0.12725 -0.068272 0.011099" rpy="0 0 0"/>
+    <origin xyz="-0.130949 -0.059914 0.011099" rpy="0 0 0"/>
     <geometry>
       <mesh filename="package://animatronics_urdf_description/meshes/XL-430_new_v5_1.stl" scale="0.001 0.001 0.001"/>
@@ -665,10 +665,10 @@
 <link name="Neck_Gear_Mid_v13_1">
   <inertial>
-    <origin xyz="-0.008793252964029358 -1.8220616238018295e-07 0.011979756069733671" rpy="0 0 0"/>
+    <origin xyz="-0.00796981243534886 0.0037159124695311796 0.011979756069755789" rpy="0 0 0"/>
     <mass value="0.14220453425486923"/>
-    <inertia ixx="3.8e-05" iyy="4.8e-05" izz="4e-05" ixy="-0.0" iyz="0.0" ixz="1.6e-05"/>
-  </inertial>
-  <visual>
-    <origin xyz="-0.12925 -0.100272 9.9e-05" rpy="0 0 0"/>
+    <inertia ixx="4e-05" iyy="4.6e-05" izz="4e-05" ixy="4e-06" iyz="-7e-06" ixz="1.4e-05"/>
+  </inertial>
+  <visual>
+    <origin xyz="-0.146286 -0.088071 9.9e-05" rpy="0 0 0"/>
     <geometry>
       <mesh filename="package://animatronics_urdf_description/meshes/Neck_Gear_Mid_v13_1.stl" scale="0.001 0.001 0.001"/>
@@ -677,5 +677,5 @@
   </visual>
   <collision>
-    <origin xyz="-0.12925 -0.100272 9.9e-05" rpy="0 0 0"/>
+    <origin xyz="-0.146286 -0.088071 9.9e-05" rpy="0 0 0"/>
     <geometry>
       <mesh filename="package://animatronics_urdf_description/meshes/Neck_Gear_Mid_v13_1.stl" scale="0.001 0.001 0.001"/>
@@ -685,10 +685,10 @@
 <link name="NeckMidGearHolder_v1_1">
   <inertial>
-    <origin xyz="-0.006000000992760157 0.010169907949410473 -0.014349853833520759" rpy="0 0 0"/>
+    <origin xyz="-0.001139674877776109 0.011752471334179337 -0.014349853833493447" rpy="0 0 0"/>
     <mass value="0.063161529786995"/>
-    <inertia ixx="1.7e-05" iyy="2.1e-05" izz="1e-05" ixy="-0.0" iyz="-0.0" ixz="0.0"/>
-  </inertial>
-  <visual>
-    <origin xyz="-0.11625 -0.096272 -0.014151" rpy="0 0 0"/>
+    <inertia ixx="1.8e-05" iyy="2e-05" izz="1e-05" ixy="1e-06" iyz="-0.0" ixz="-0.0"/>
+  </inertial>
+  <visual>
+    <origin xyz="-0.132813 -0.08994 -0.014151" rpy="0 0 0"/>
     <geometry>
       <mesh filename="package://animatronics_urdf_description/meshes/NeckMidGearHolder_v1_1.stl" scale="0.001 0.001 0.001"/>
@@ -697,5 +697,5 @@
   </visual>
   <collision>
-    <origin xyz="-0.11625 -0.096272 -0.014151" rpy="0 0 0"/>
+    <origin xyz="-0.132813 -0.08994 -0.014151" rpy="0 0 0"/>
     <geometry>
       <mesh filename="package://animatronics_urdf_description/meshes/NeckMidGearHolder_v1_1.stl" scale="0.001 0.001 0.001"/>
@@ -705,10 +705,10 @@
 <link name="Neck_Gear_Mid_Axis_v6_1">
   <inertial>
-    <origin xyz="7.809586310969507e-13 -0.0005357886973757497 1.6284542379155025e-07" rpy="0 0 0"/>
+    <origin xyz="-0.00022631360814251433 -0.0004850682089249242 1.6284545517670948e-07" rpy="0 0 0"/>
     <mass value="0.02076155413049806"/>
-    <inertia ixx="1e-06" iyy="2e-06" izz="1e-06" ixy="-0.0" iyz="0.0" ixz="-0.0"/>
-  </inertial>
-  <visual>
-    <origin xyz="-0.11025 -0.114522 0.000199" rpy="0 0 0"/>
+    <inertia ixx="1e-06" iyy="2e-06" izz="1e-06" ixy="0.0" iyz="0.0" ixz="0.0"/>
+  </inertial>
+  <visual>
+    <origin xyz="-0.135088 -0.109015 0.000199" rpy="0 0 0"/>
     <geometry>
       <mesh filename="package://animatronics_urdf_description/meshes/Neck_Gear_Mid_Axis_v6_1.stl" scale="0.001 0.001 0.001"/>
@@ -717,5 +717,5 @@
   </visual>
   <collision>
-    <origin xyz="-0.11025 -0.114522 0.000199" rpy="0 0 0"/>
+    <origin xyz="-0.135088 -0.109015 0.000199" rpy="0 0 0"/>
     <geometry>
       <mesh filename="package://animatronics_urdf_description/meshes/Neck_Gear_Mid_Axis_v6_1.stl" scale="0.001 0.001 0.001"/>
@@ -725,10 +725,10 @@
 <link name="Neck_Gear_Top_v17_1">
   <inertial>
-    <origin xyz="1.7835116590536604e-07 0.004768131192007488 0.00523945488896141" rpy="0 0 0"/>
+    <origin xyz="0.0020152362214851116 0.004321763675619095 0.005239454888997268" rpy="0 0 0"/>
     <mass value="0.325166045089014"/>
-    <inertia ixx="0.000186" iyy="0.000113" izz="0.000133" ixy="-0.0" iyz="3.9e-05" ixz="-0.0"/>
-  </inertial>
-  <visual>
-    <origin xyz="-0.11025 -0.117522 0.000199" rpy="0 0 0"/>
+    <inertia ixx="0.000173" iyy="0.000126" izz="0.000133" ixy="-2.8e-05" iyz="3.5e-05" ixz="1.6e-05"/>
+  </inertial>
+  <visual>
+    <origin xyz="-0.136356 -0.111734 0.000199" rpy="0 0 0"/>
     <geometry>
       <mesh filename="package://animatronics_urdf_description/meshes/Neck_Gear_Top_v17_1.stl" scale="0.001 0.001 0.001"/>
@@ -737,5 +737,5 @@
   </visual>
   <collision>
-    <origin xyz="-0.11025 -0.117522 0.000199" rpy="0 0 0"/>
+    <origin xyz="-0.136356 -0.111734 0.000199" rpy="0 0 0"/>
     <geometry>
       <mesh filename="package://animatronics_urdf_description/meshes/Neck_Gear_Top_v17_1.stl" scale="0.001 0.001 0.001"/>
@@ -745,10 +745,10 @@
 <link name="2XC-430_v6_1">
   <inertial>
-    <origin xyz="3.889727131396736e-05 0.011999704196970246 -0.01903867982801462" rpy="0 0 0"/>
+    <origin xyz="3.8730834067995934e-05 0.012000459371747318 -0.019038679827954846" rpy="0 0 0"/>
     <mass value="0.09031899704975468"/>
     <inertia ixx="2.7e-05" iyy="2.3e-05" izz="2.7e-05" ixy="0.0" iyz="0.0" ixz="0.0"/>
   </inertial>
   <visual>
-    <origin xyz="-0.11025 -0.166616 -0.018801" rpy="0 0 0"/>
+    <origin xyz="-0.157104 -0.156228 -0.018801" rpy="0 0 0"/>
     <geometry>
       <mesh filename="package://animatronics_urdf_description/meshes/2XC-430_v6_1.stl" scale="0.001 0.001 0.001"/>
@@ -757,5 +757,5 @@
   </visual>
   <collision>
-    <origin xyz="-0.11025 -0.166616 -0.018801" rpy="0 0 0"/>
+    <origin xyz="-0.157104 -0.156228 -0.018801" rpy="0 0 0"/>
     <geometry>
       <mesh filename="package://animatronics_urdf_description/meshes/2XC-430_v6_1.stl" scale="0.001 0.001 0.001"/>
@@ -765,10 +765,10 @@
 <link name="Head_Joint_v6_1">
   <inertial>
-    <origin xyz="0.03210680929658477 0.007684916074679304 1.6788690773629922e-07" rpy="0 0 0"/>
+    <origin xyz="0.032106642859338674 0.007685671249456377 1.6788696751454495e-07" rpy="0 0 0"/>
     <mass value="0.01706262563442855"/>
     <inertia ixx="8e-06" iyy="1.1e-05" izz="8e-06" ixy="2e-06" iyz="0.0" ixz="-0.0"/>
   </inertial>
   <visual>
-    <origin xyz="-0.09125 -0.190616 0.000199" rpy="0 0 0"/>
+    <origin xyz="-0.138104 -0.180228 0.000199" rpy="0 0 0"/>
     <geometry>
       <mesh filename="package://animatronics_urdf_description/meshes/Head_Joint_v6_1.stl" scale="0.001 0.001 0.001"/>
@@ -777,5 +777,5 @@
   </visual>
   <collision>
-    <origin xyz="-0.09125 -0.190616 0.000199" rpy="0 0 0"/>
+    <origin xyz="-0.138104 -0.180228 0.000199" rpy="0 0 0"/>
     <geometry>
       <mesh filename="package://animatronics_urdf_description/meshes/Head_Joint_v6_1.stl" scale="0.001 0.001 0.001"/>
@@ -785,10 +785,10 @@
 <link name="Head_MainPlate_v4_1">
   <inertial>
-    <origin xyz="0.06759705203616215 -0.0025007283450097506 0.02869529974461484" rpy="0 0 0"/>
+    <origin xyz="0.06759688559891597 -0.0024999731702323724 0.028695299744674618" rpy="0 0 0"/>
     <mass value="0.4432124636647733"/>
     <inertia ixx="0.000151" iyy="0.000889" izz="0.000755" ixy="4e-06" iyz="0.0" ixz="6e-06"/>
   </inertial>
   <visual>
-    <origin xyz="-0.13475 -0.176616 0.028699" rpy="0 0 0"/>
+    <origin xyz="-0.181604 -0.166228 0.028699" rpy="0 0 0"/>
     <geometry>
       <mesh filename="package://animatronics_urdf_description/meshes/Head_MainPlate_v4_1.stl" scale="0.001 0.001 0.001"/>
@@ -797,5 +797,5 @@
   </visual>
   <collision>
-    <origin xyz="-0.13475 -0.176616 0.028699" rpy="0 0 0"/>
+    <origin xyz="-0.181604 -0.166228 0.028699" rpy="0 0 0"/>
     <geometry>
       <mesh filename="package://animatronics_urdf_description/meshes/Head_MainPlate_v4_1.stl" scale="0.001 0.001 0.001"/>
@@ -805,10 +805,10 @@
 <link name="XL-430_new_v5_2">
   <inertial>
-    <origin xyz="0.020332582443741226 -0.011008502903220196 -0.01766572164346647" rpy="0 0 0"/>
+    <origin xyz="0.020332416006495213 -0.011007747728442957 -0.017665721643406695" rpy="0 0 0"/>
     <mass value="0.33677880262575866"/>
     <inertia ixx="5.5e-05" iyy="9.4e-05" izz="8.2e-05" ixy="0.0" iyz="-0.0" ixz="0.0"/>
   </inertial>
   <visual>
-    <origin xyz="-0.13375 -0.167116 -0.016801" rpy="0 0 0"/>
+    <origin xyz="-0.180604 -0.156728 -0.016801" rpy="0 0 0"/>
     <geometry>
       <mesh filename="package://animatronics_urdf_description/meshes/XL-430_new_v5_2.stl" scale="0.001 0.001 0.001"/>
@@ -817,5 +817,5 @@
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