Commit message: fix urdf names for isaac sim compatibility

File: animatronics_urdf_description/animatronics_urdf_description_standalone.urdf (robot description, URDF)
Before this commit: robot urdf, 48 links, 47 joints
Links:
- removed link 2XC-430_v6_1
- removed link 51202_v2_1
- removed link 51202_v2_2
- removed link 51202_v2_3
- removed link 51202_v2_4
- removed link 51202_v2_5
- removed link 51202_v2_6
- removed link 6900ZZNR_v2_1
- removed link 6900ZZNR_v2_2
- removed link XL-430_new_v5_1
- removed link XL-430_new_v5_2
- removed link XM,H,D-540.N101.I101_v5_1
- removed link XM,H,D-540.N101.I101_v5_2
- removed link XM,H,D-540.N101.I101_v5_3
- removed link XM,H,D-540.N101.I101_v5_4
- removed link XM,H,D-540.N101.I101_v5_5
- removed link XM,H,D-540.N101.I101_v5_6
- removed link XM,H,D-540.N101.I101_v5_7
- removed link XM,H,D-540.N101.I101_v5_8
- removed link XM,H-430_idler_v3_1
- added link Link_2XC_430_v6_1, mass 0.09031899704975468; collision mesh filename=./meshes/Link_2XC_430_v6_1.stl scale=0.001 0.001 0.001; visual mesh filename=./meshes/Link_2XC_430_v6_1.stl scale=0.001 0.001 0.001
- added link Link_51202_v2_1, mass 0.05505680395324213; collision mesh filename=./meshes/Link_51202_v2_1.stl scale=0.001 0.001 0.001; visual mesh filename=./meshes/Link_51202_v2_1.stl scale=0.001 0.001 0.001
- added link Link_51202_v2_2, mass 0.05505680395324213; collision mesh filename=./meshes/Link_51202_v2_2.stl scale=0.001 0.001 0.001; visual mesh filename=./meshes/Link_51202_v2_2.stl scale=0.001 0.001 0.001
- added link Link_51202_v2_3, mass 0.05505680395324213; collision mesh filename=./meshes/Link_51202_v2_3.stl scale=0.001 0.001 0.001; visual mesh filename=./meshes/Link_51202_v2_3.stl scale=0.001 0.001 0.001
- added link Link_51202_v2_4, mass 0.05505680395324213; collision mesh filename=./meshes/Link_51202_v2_4.stl scale=0.001 0.001 0.001; visual mesh filename=./meshes/Link_51202_v2_4.stl scale=0.001 0.001 0.001
- added link Link_51202_v2_5, mass 0.05505680395324213; collision mesh filename=./meshes/Link_51202_v2_5.stl scale=0.001 0.001 0.001; visual mesh filename=./meshes/Link_51202_v2_5.stl scale=0.001 0.001 0.001
- added link Link_51202_v2_6, mass 0.05505680395324213; collision mesh filename=./meshes/Link_51202_v2_6.stl scale=0.001 0.001 0.001; visual mesh filename=./meshes/Link_51202_v2_6.stl scale=0.001 0.001 0.001
- added link Link_6900ZZNR_v2_1, mass 0.014205025342471455; collision mesh filename=./meshes/Link_6900ZZNR_v2_1.stl scale=0.001 0.001 0.001; visual mesh filename=./meshes/Link_6900ZZNR_v2_1.stl scale=0.001 0.001 0.001
- added link Link_6900ZZNR_v2_2, mass 0.014205025342471455; collision mesh filename=./meshes/Link_6900ZZNR_v2_2.stl scale=0.001 0.001 0.001; visual mesh filename=./meshes/Link_6900ZZNR_v2_2.stl scale=0.001 0.001 0.001
- added link XL_430_new_v5_1, mass 0.33677880262575866; collision mesh filename=./meshes/XL_430_new_v5_1.stl scale=0.001 0.001 0.001; visual mesh filename=./meshes/XL_430_new_v5_1.stl scale=0.001 0.001 0.001
- added link XL_430_new_v5_2, mass 0.33677880262575866; collision mesh filename=./meshes/XL_430_new_v5_2.stl scale=0.001 0.001 0.001; visual mesh filename=./meshes/XL_430_new_v5_2.stl scale=0.001 0.001 0.001
- added link XM_H_430_idler_v3_1, mass 0.12871928366116375; collision mesh filename=./meshes/XM_H_430_idler_v3_1.stl scale=0.001 0.001 0.001; visual mesh filename=./meshes/XM_H_430_idler_v3_1.stl scale=0.001 0.001 0.001
- added link XM_H_D_540_N101_I101_v5_1, mass 0.6640277986148612; collision mesh filename=./meshes/XM_H_D_540_N101_I101_v5_1.stl scale=0.001 0.001 0.001; visual mesh filename=./meshes/XM_H_D_540_N101_I101_v5_1.stl scale=0.001 0.001 0.001
- added link XM_H_D_540_N101_I101_v5_2, mass 0.6640277986148612; collision mesh filename=./meshes/XM_H_D_540_N101_I101_v5_2.stl scale=0.001 0.001 0.001; visual mesh filename=./meshes/XM_H_D_540_N101_I101_v5_2.stl scale=0.001 0.001 0.001
- added link XM_H_D_540_N101_I101_v5_3, mass 0.6640277986148612; collision mesh filename=./meshes/XM_H_D_540_N101_I101_v5_3.stl scale=0.001 0.001 0.001; visual mesh filename=./meshes/XM_H_D_540_N101_I101_v5_3.stl scale=0.001 0.001 0.001
- added link XM_H_D_540_N101_I101_v5_4, mass 0.6640277986148612; collision mesh filename=./meshes/XM_H_D_540_N101_I101_v5_4.stl scale=0.001 0.001 0.001; visual mesh filename=./meshes/XM_H_D_540_N101_I101_v5_4.stl scale=0.001 0.001 0.001
- added link XM_H_D_540_N101_I101_v5_5, mass 0.6640277986148612; collision mesh filename=./meshes/XM_H_D_540_N101_I101_v5_5.stl scale=0.001 0.001 0.001; visual mesh filename=./meshes/XM_H_D_540_N101_I101_v5_5.stl scale=0.001 0.001 0.001
- added link XM_H_D_540_N101_I101_v5_6, mass 0.6640277986148612; collision mesh filename=./meshes/XM_H_D_540_N101_I101_v5_6.stl scale=0.001 0.001 0.001; visual mesh filename=./meshes/XM_H_D_540_N101_I101_v5_6.stl scale=0.001 0.001 0.001
- added link XM_H_D_540_N101_I101_v5_7, mass 0.6640277986148612; collision mesh filename=./meshes/XM_H_D_540_N101_I101_v5_7.stl scale=0.001 0.001 0.001; visual mesh filename=./meshes/XM_H_D_540_N101_I101_v5_7.stl scale=0.001 0.001 0.001
- added link XM_H_D_540_N101_I101_v5_8, mass 0.6640277986148612; collision mesh filename=./meshes/XM_H_D_540_N101_I101_v5_8.stl scale=0.001 0.001 0.001; visual mesh filename=./meshes/XM_H_D_540_N101_I101_v5_8.stl scale=0.001 0.001 0.001
- link Head_Joint_v6_1: geometry collision mesh filename=./meshes/Head_Joint_v6_1.stl scale=0.001 0.001 0.001; visual mesh filename=./meshes/Head_Joint_v6_1.stl scale=0.001 0.001 0.001
- link Head_MainPlate_v4_1: geometry collision mesh filename=./meshes/Head_MainPlate_v4_1.stl scale=0.001 0.001 0.001; visual mesh filename=./meshes/Head_MainPlate_v4_1.stl scale=0.001 0.001 0.001
- link Jaw_v4_1: geometry collision mesh filename=./meshes/Jaw_v4_1.stl scale=0.001 0.001 0.001; visual mesh filename=./meshes/Jaw_v4_1.stl scale=0.001 0.001 0.001
- link Leg01_v11_1: geometry collision mesh filename=./meshes/Leg01_v11_1.stl scale=0.001 0.001 0.001; visual mesh filename=./meshes/Leg01_v11_1.stl scale=0.001 0.001 0.001
- link Leg01_v11_2: geometry collision mesh filename=./meshes/Leg01_v11_2.stl scale=0.001 0.001 0.001; visual mesh filename=./meshes/Leg01_v11_2.stl scale=0.001 0.001 0.001
- link Leg02_v10_1: geometry collision mesh filename=./meshes/Leg02_v10_1.stl scale=0.001 0.001 0.001; visual mesh filename=./meshes/Leg02_v10_1.stl scale=0.001 0.001 0.001
- link Leg02_v10_2: geometry collision mesh filename=./meshes/Leg02_v10_2.stl scale=0.001 0.001 0.001; visual mesh filename=./meshes/Leg02_v10_2.stl scale=0.001 0.001 0.001
- link Leg03_v28_1: geometry collision mesh filename=./meshes/Leg03_v28_1.stl scale=0.001 0.001 0.001; visual mesh filename=./meshes/Leg03_v28_1.stl scale=0.001 0.001 0.001
- link Leg03_v28_2: geometry collision mesh filename=./meshes/Leg03_v28_2.stl scale=0.001 0.001 0.001; visual mesh filename=./meshes/Leg03_v28_2.stl scale=0.001 0.001 0.001
- link Leg04_v11_1: geometry collision mesh filename=./meshes/Leg04_v11_1.stl scale=0.001 0.001 0.001; visual mesh filename=./meshes/Leg04_v11_1.stl scale=0.001 0.001 0.001
- link Leg04_v11_2: geometry collision mesh filename=./meshes/Leg04_v11_2.stl scale=0.001 0.001 0.001; visual mesh filename=./meshes/Leg04_v11_2.stl scale=0.001 0.001 0.001
- link Leg_Cover_v3_1: geometry collision mesh filename=./meshes/Leg_Cover_v3_1.stl scale=0.001 0.001 0.001; visual mesh filename=./meshes/Leg_Cover_v3_1.stl scale=0.001 0.001 0.001
- link Leg_Cover_v3_2: geometry collision mesh filename=./meshes/Leg_Cover_v3_2.stl scale=0.001 0.001 0.001; visual mesh filename=./meshes/Leg_Cover_v3_2.stl scale=0.001 0.001 0.001
- link Leg_Rotator_Upper_v4_1: geometry collision mesh filename=./meshes/Leg_Rotator_Upper_v4_1.stl scale=0.001 0.001 0.001; visual mesh filename=./meshes/Leg_Rotator_Upper_v4_1.stl scale=0.001 0.001 0.001
- link Leg_Rotator_Upper_v4_2: geometry collision mesh filename=./meshes/Leg_Rotator_Upper_v4_2.stl scale=0.001 0.001 0.001; visual mesh filename=./meshes/Leg_Rotator_Upper_v4_2.stl scale=0.001 0.001 0.001
- link Leg_Rotator_v10_1: geometry collision mesh filename=./meshes/Leg_Rotator_v10_1.stl scale=0.001 0.001 0.001; visual mesh filename=./meshes/Leg_Rotator_v10_1.stl scale=0.001 0.001 0.001
- link Leg_Rotator_v10_2: geometry collision mesh filename=./meshes/Leg_Rotator_v10_2.stl scale=0.001 0.001 0.001; visual mesh filename=./meshes/Leg_Rotator_v10_2.stl scale=0.001 0.001 0.001
- link NeckMidGearHolder_v1_1: geometry collision mesh filename=./meshes/NeckMidGearHolder_v1_1.stl scale=0.001 0.001 0.001; visual mesh filename=./meshes/NeckMidGearHolder_v1_1.stl scale=0.001 0.001 0.001
- link Neck_Bar_v1_1: geometry collision mesh filename=./meshes/Neck_Bar_v1_1.stl scale=0.001 0.001 0.001; visual mesh filename=./meshes/Neck_Bar_v1_1.stl scale=0.001 0.001 0.001
- link Neck_Bar_v1_2: geometry collision mesh filename=./meshes/Neck_Bar_v1_2.stl scale=0.001 0.001 0.001; visual mesh filename=./meshes/Neck_Bar_v1_2.stl scale=0.001 0.001 0.001
- link Neck_Gear_Mid_Axis_v6_1: geometry collision mesh filename=./meshes/Neck_Gear_Mid_Axis_v6_1.stl scale=0.001 0.001 0.001; visual mesh filename=./meshes/Neck_Gear_Mid_Axis_v6_1.stl scale=0.001 0.001 0.001
- link Neck_Gear_Mid_v13_1: geometry collision mesh filename=./meshes/Neck_Gear_Mid_v13_1.stl scale=0.001 0.001 0.001; visual mesh filename=./meshes/Neck_Gear_Mid_v13_1.stl scale=0.001 0.001 0.001
- link Neck_Gear_Top_v17_1: geometry collision mesh filename=./meshes/Neck_Gear_Top_v17_1.stl scale=0.001 0.001 0.001; visual mesh filename=./meshes/Neck_Gear_Top_v17_1.stl scale=0.001 0.001 0.001
- link Neck_Gear_v10_1: geometry collision mesh filename=./meshes/Neck_Gear_v10_1.stl scale=0.001 0.001 0.001; visual mesh filename=./meshes/Neck_Gear_v10_1.stl scale=0.001 0.001 0.001
- link Neck_JointH_v28_1: geometry collision mesh filename=./meshes/Neck_JointH_v28_1.stl scale=0.001 0.001 0.001; visual mesh filename=./meshes/Neck_JointH_v28_1.stl scale=0.001 0.001 0.001
- link Tail_Base_v3_1: geometry collision mesh filename=./meshes/Tail_Base_v3_1.stl scale=0.001 0.001 0.001; visual mesh filename=./meshes/Tail_Base_v3_1.stl scale=0.001 0.001 0.001
- link base_link: geometry collision mesh filename=./meshes/base_link.stl scale=0.001 0.001 0.001; visual mesh filename=./meshes/base_link.stl scale=0.001 0.001 0.001
- link body_cover_v21_1: geometry collision mesh filename=./meshes/body_cover_v21_1.stl scale=0.001 0.001 0.001; visual mesh filename=./meshes/body_cover_v21_1.stl scale=0.001 0.001 0.001
Joints:
- removed joint Revolute 10
- removed joint Revolute 12
- removed joint Revolute 13
- removed joint Revolute 16
- removed joint Revolute 17
- removed joint Revolute 20
- removed joint Revolute 22
- removed joint Revolute 23
- removed joint Revolute 26
- removed joint Revolute 27
- removed joint Revolute 37
- removed joint Revolute 42
- removed joint Revolute 43
- removed joint Revolute 44
- removed joint Rigid 11
- removed joint Rigid 14
- removed joint Rigid 15
- removed joint Rigid 18
- removed joint Rigid 19
- removed joint Rigid 21
- removed joint Rigid 24
- removed joint Rigid 25
- removed joint Rigid 28
- removed joint Rigid 29
- removed joint Rigid 30
- removed joint Rigid 31
- removed joint Rigid 32
- removed joint Rigid 33
- removed joint Rigid 34
- removed joint Rigid 36
- removed joint Rigid 38
- removed joint Rigid 39
- removed joint Rigid 40
- removed joint Rigid 41
- removed joint Rigid 45
- removed joint Rigid 46
- removed joint Rigid 47
- removed joint Rigid 48
- removed joint Rigid 49
- removed joint Rigid 50
- removed joint Rigid 51
- removed joint Rigid 52
- removed joint Rigid 58
- removed joint Rigid 6
- removed joint Rigid 7
- removed joint Rigid 8
- removed joint Rigid 9
- added joint Revolute_10: type continuous, parent Link_51202_v2_1, child Leg_Rotator_v10_1, origin xyz=0.0 0.012 0.0 rpy=0 0 0, axis 0.0 1.0 0.0
- added joint Revolute_12: type continuous, parent XM_H_D_540_N101_I101_v5_1, child Leg01_v11_1, origin xyz=0.0165 0.038 -0.01675 rpy=0 0 0, axis -1.0 0.0 0.0
- added joint Revolute_13: type continuous, parent Leg01_v11_1, child XM_H_D_540_N101_I101_v5_2, origin xyz=-0.0245 -0.0135 0.084 rpy=0 0 0, axis 0.0 0.0 -1.0
- added joint Revolute_16: type continuous, parent XM_H_D_540_N101_I101_v5_3, child Leg03_v28_1, origin xyz=0.018343 -0.037257 0.0165 rpy=0 0 0, axis -0.0 0.0 -1.0
- added joint Revolute_17: type continuous, parent Leg03_v28_1, child XM_H_D_540_N101_I101_v5_4, origin xyz=-0.077135 -0.091926 0.0 rpy=0 0 0, axis -0.0 0.0 -1.0
- added joint Revolute_20: type continuous, parent Link_51202_v2_2, child Leg_Rotator_v10_2, origin xyz=0.0 0.012 0.0 rpy=0 0 0, axis 0.0 1.0 0.0
- added joint Revolute_22: type continuous, parent XM_H_D_540_N101_I101_v5_5, child Leg01_v11_2, origin xyz=0.0165 0.038 -0.01675 rpy=0 0 0, axis -1.0 0.0 0.0
- added joint Revolute_23: type continuous, parent Leg01_v11_2, child XM_H_D_540_N101_I101_v5_6, origin xyz=-0.0245 -0.0135 -0.084 rpy=0 0 0, axis 0.0 -0.0 1.0
- added joint Revolute_26: type continuous, parent XM_H_D_540_N101_I101_v5_7, child Leg03_v28_2, origin xyz=0.039877 -0.011594 -0.0325 rpy=0 0 0, axis -0.0 -0.0 1.0
- added joint Revolute_27: type continuous, parent Leg03_v28_2, child XM_H_D_540_N101_I101_v5_8, origin xyz=-0.077135 -0.091926 0.0 rpy=0 0 0, axis 0.0 -0.0 1.0
- added joint Revolute_37: type continuous, parent base_link, child Link_6900ZZNR_v2_1, origin xyz=0.11025 0.05575 0.0215 rpy=0 0 0, axis -0.0 -0.0 1.0
- added joint Revolute_42: type continuous, parent Neck_Gear_Mid_Axis_v6_1, child Neck_Gear_Top_v17_1, origin xyz=0.001268 0.002719 0.0 rpy=0 0 0, axis -0.422618 -0.906308 -0.0
- added joint Revolute_43: type continuous, parent Neck_Gear_Top_v17_1, child Link_2XC_430_v6_1, origin xyz=0.020748 0.044494 0.019 rpy=0 0 0, axis 0.0 0.0 -1.0
- added joint Revolute_44: type continuous, parent Link_2XC_430_v6_1, child Head_Joint_v6_1, origin xyz=-0.019 0.024 -0.019 rpy=0 0 0, axis -1.0 -0.0 -0.0
- added joint Rigid_11: type fixed, parent Leg_Rotator_v10_1, child XM_H_D_540_N101_I101_v5_1, origin xyz=0.008 0.01175 0.01675 rpy=0 0 0
- added joint Rigid_14: type fixed, parent XM_H_D_540_N101_I101_v5_2, child Leg02_v10_1, origin xyz=0.018343 -0.037257 -0.0165 rpy=0 0 0
- added joint Rigid_15: type fixed, parent Leg02_v10_1, child XM_H_D_540_N101_I101_v5_3, origin xyz=0.115374 -0.053079 0.0 rpy=0 0 0
- added joint Rigid_18: type fixed, parent XM_H_D_540_N101_I101_v5_4, child Leg04_v11_1, origin xyz=0.035517 -0.02152 -0.0165 rpy=0 0 0
- added joint Rigid_19: type fixed, parent Leg04_v11_1, child Leg_Cover_v3_1, origin xyz=0.00984 -0.06775 -0.021716 rpy=0 0 0
- added joint Rigid_21: type fixed, parent Leg_Rotator_v10_2, child XM_H_D_540_N101_I101_v5_5, origin xyz=0.008 0.01175 0.01675 rpy=0 0 0
- added joint Rigid_24: type fixed, parent XM_H_D_540_N101_I101_v5_6, child Leg02_v10_2, origin xyz=0.018343 -0.037257 0.0325 rpy=0 0 0
- added joint Rigid_25: type fixed, parent Leg02_v10_2, child XM_H_D_540_N101_I101_v5_7, origin xyz=0.09384 -0.078742 0.0 rpy=0 0 0
- added joint Rigid_28: type fixed, parent XM_H_D_540_N101_I101_v5_8, child Leg04_v11_2, origin xyz=0.035517 -0.02152 0.0165 rpy=0 0 0
- added joint Rigid_29: type fixed, parent Leg04_v11_2, child Leg_Cover_v3_2, origin xyz=0.00984 -0.06775 0.021716 rpy=0 0 0
- added joint Rigid_30: type fixed, parent base_link, child Tail_Base_v3_1, origin xyz=-0.13 -0.026 -0.035 rpy=0 0 0
- added joint Rigid_31: type fixed, parent base_link, child XM_H_430_idler_v3_1, origin xyz=0.117 0.00325 -0.0215 rpy=0 0 0
- added joint Rigid_32: type fixed, parent XM_H_430_idler_v3_1, child Neck_Gear_v10_1, origin xyz=-0.008 0.011 0.036 rpy=0 0 0
- added joint Rigid_33: type fixed, parent base_link, child Neck_Bar_v1_1, origin xyz=0.117466 0.05875 -0.0315 rpy=0 0 0
- added joint Rigid_34: type fixed, parent base_link, child Neck_Bar_v1_2, origin xyz=0.11725 0.05275 0.0315 rpy=0 0 0
- added joint Rigid_36: type fixed, parent Neck_JointH_v28_1, child Link_6900ZZNR_v2_2, origin xyz=0.0 0.0 -0.031 rpy=0 0 0
- added joint Rigid_38: type fixed, parent Neck_JointH_v28_1, child XL_430_new_v5_1, origin xyz=0.020699 0.004164 -0.026599 rpy=0 0 0
- added joint Rigid_39: type fixed, parent XL_430_new_v5_1, child Neck_Gear_Mid_v13_1, origin xyz=0.015337 0.028157 0.011 rpy=0 0 0
- added joint Rigid_40: type fixed, parent XL_430_new_v5_1, child NeckMidGearHolder_v1_1, origin xyz=0.001864 0.030026 0.02525 rpy=0 0 0
- added joint Rigid_41: type fixed, parent NeckMidGearHolder_v1_1, child Neck_Gear_Mid_Axis_v6_1, origin xyz=0.002275 0.019075 -0.01435 rpy=0 0 0
- added joint Rigid_45: type fixed, parent Head_Joint_v6_1, child Head_MainPlate_v4_1, origin xyz=0.0435 -0.014 -0.0285 rpy=0 0 0
- added joint Rigid_46: type fixed, parent Head_MainPlate_v4_1, child XL_430_new_v5_2, origin xyz=-0.001 -0.0095 0.0455 rpy=0 0 0
- added joint Rigid_47: type fixed, parent XL_430_new_v5_2, child Jaw_v4_1, origin xyz=0.032 -0.011 -0.036 rpy=0 0 0
- added joint Rigid_48: type fixed, parent Link_6900ZZNR_v2_1, child Neck_JointH_v28_1, origin xyz=0.0 0.0 -0.006 rpy=0 0 0
- added joint Rigid_49: type fixed, parent XM_H_D_540_N101_I101_v5_1, child Leg_Rotator_Upper_v4_1, origin xyz=0.0 0.032 0.0 rpy=0 0 0
- added joint Rigid_50: type fixed, parent Leg_Rotator_Upper_v4_1, child Link_51202_v2_5, origin xyz=-0.008 0.02375 -0.01675 rpy=0 0 0
- added joint Rigid_51: type fixed, parent XM_H_D_540_N101_I101_v5_5, child Leg_Rotator_Upper_v4_2, origin xyz=0.0 0.032 0.0 rpy=0 0 0
- added joint Rigid_52: type fixed, parent Leg_Rotator_Upper_v4_2, child Link_51202_v2_6, origin xyz=-0.008 0.02375 -0.01675 rpy=0 0 0
- added joint Rigid_58: type fixed, parent base_link, child body_cover_v21_1, origin xyz=-0.125 0.0385 0.0 rpy=0 0 0
- added joint Rigid_6: type fixed, parent base_link, child Link_51202_v2_1, origin xyz=-0.099 -0.011 0.0705 rpy=0 0 0
- added joint Rigid_7: type fixed, parent base_link, child Link_51202_v2_2, origin xyz=-0.099 -0.011 -0.0705 rpy=0 0 0
- added joint Rigid_8: type fixed, parent base_link, child Link_51202_v2_3, origin xyz=-0.033 -0.011 -0.0705 rpy=0 0 0
- added joint Rigid_9: type fixed, parent base_link, child Link_51202_v2_4, origin xyz=-0.033 -0.011 0.0705 rpy=0 0 0
