Commit message: fix urdf names for isaac sim compatibility

File: animatronics_urdf_description/urdf/animatronics_urdf.xacro (robot description, xacro)
@@ -23,5 +23,5 @@
   </collision>
 </link>
-<link name="51202_v2_1">
+<link name="Link_51202_v2_1">
   <inertial>
     <origin xyz="-2.674484661513432e-10 0.005999999999999998 9.590508942558529e-12" rpy="0 0 0"/>
@@ -32,5 +32,5 @@
     <origin xyz="0.099 0.011 -0.0705" rpy="0 0 0"/>
     <geometry>
-      <mesh filename="package://animatronics_urdf_description/meshes/51202_v2_1.stl" scale="0.001 0.001 0.001"/>
+      <mesh filename="package://animatronics_urdf_description/meshes/Link_51202_v2_1.stl" scale="0.001 0.001 0.001"/>
     </geometry>
     <material name="steel_satin"/>
@@ -39,9 +39,9 @@
     <origin xyz="0.099 0.011 -0.0705" rpy="0 0 0"/>
     <geometry>
-      <mesh filename="package://animatronics_urdf_description/meshes/51202_v2_1.stl" scale="0.001 0.001 0.001"/>
-    </geometry>
-  </collision>
-</link>
-<link name="51202_v2_2">
+      <mesh filename="package://animatronics_urdf_description/meshes/Link_51202_v2_1.stl" scale="0.001 0.001 0.001"/>
+    </geometry>
+  </collision>
+</link>
+<link name="Link_51202_v2_2">
   <inertial>
     <origin xyz="-2.764975609581555e-10 0.005999999999999998 -1.5566548050571782e-11" rpy="0 0 0"/>
@@ -52,5 +52,5 @@
     <origin xyz="0.099 0.011 0.0705" rpy="0 0 0"/>
     <geometry>
-      <mesh filename="package://animatronics_urdf_description/meshes/51202_v2_2.stl" scale="0.001 0.001 0.001"/>
+      <mesh filename="package://animatronics_urdf_description/meshes/Link_51202_v2_2.stl" scale="0.001 0.001 0.001"/>
     </geometry>
     <material name="steel_satin"/>
@@ -59,9 +59,9 @@
     <origin xyz="0.099 0.011 0.0705" rpy="0 0 0"/>
     <geometry>
-      <mesh filename="package://animatronics_urdf_description/meshes/51202_v2_2.stl" scale="0.001 0.001 0.001"/>
-    </geometry>
-  </collision>
-</link>
-<link name="51202_v2_3">
+      <mesh filename="package://animatronics_urdf_description/meshes/Link_51202_v2_2.stl" scale="0.001 0.001 0.001"/>
+    </geometry>
+  </collision>
+</link>
+<link name="Link_51202_v2_3">
   <inertial>
     <origin xyz="-2.8593932083209594e-10 0.005999999999999998 2.916361596660977e-12" rpy="0 0 0"/>
@@ -72,5 +72,5 @@
     <origin xyz="0.033 0.011 0.0705" rpy="0 0 0"/>
     <geometry>
-      <mesh filename="package://animatronics_urdf_description/meshes/51202_v2_3.stl" scale="0.001 0.001 0.001"/>
+      <mesh filename="package://animatronics_urdf_description/meshes/Link_51202_v2_3.stl" scale="0.001 0.001 0.001"/>
     </geometry>
     <material name="steel_satin"/>
@@ -79,9 +79,9 @@
     <origin xyz="0.033 0.011 0.0705" rpy="0 0 0"/>
     <geometry>
-      <mesh filename="package://animatronics_urdf_description/meshes/51202_v2_3.stl" scale="0.001 0.001 0.001"/>
-    </geometry>
-  </collision>
-</link>
-<link name="51202_v2_4">
+      <mesh filename="package://animatronics_urdf_description/meshes/Link_51202_v2_3.stl" scale="0.001 0.001 0.001"/>
+    </geometry>
+  </collision>
+</link>
+<link name="Link_51202_v2_4">
   <inertial>
     <origin xyz="-2.7689021214749587e-10 0.005999999999999998 -1.7363888105137448e-11" rpy="0 0 0"/>
@@ -92,5 +92,5 @@
     <origin xyz="0.033 0.011 -0.0705" rpy="0 0 0"/>
     <geometry>
-      <mesh filename="package://animatronics_urdf_description/meshes/51202_v2_4.stl" scale="0.001 0.001 0.001"/>
+      <mesh filename="package://animatronics_urdf_description/meshes/Link_51202_v2_4.stl" scale="0.001 0.001 0.001"/>
     </geometry>
     <material name="steel_satin"/>
@@ -99,5 +99,5 @@
     <origin xyz="0.033 0.011 -0.0705" rpy="0 0 0"/>
     <geometry>
-      <mesh filename="package://animatronics_urdf_description/meshes/51202_v2_4.stl" scale="0.001 0.001 0.001"/>
+      <mesh filename="package://animatronics_urdf_description/meshes/Link_51202_v2_4.stl" scale="0.001 0.001 0.001"/>
     </geometry>
   </collision>
@@ -123,5 +123,5 @@
   </collision>
 </link>
-<link name="XM,H,D-540.N101.I101_v5_1">
+<link name="XM_H_D_540_N101_I101_v5_1">
   <inertial>
     <origin xyz="-0.007318332020298274 0.022971414590661272 -0.01674999999044581" rpy="0 0 0"/>
@@ -132,5 +132,5 @@
     <origin xyz="0.091 -0.01275 -0.08725" rpy="0 0 0"/>
     <geometry>
-      <mesh filename="package://animatronics_urdf_description/meshes/XM,H,D-540.N101.I101_v5_1.stl" scale="0.001 0.001 0.001"/>
+      <mesh filename="package://animatronics_urdf_description/meshes/XM_H_D_540_N101_I101_v5_1.stl" scale="0.001 0.001 0.001"/>
     </geometry>
     <material name="coating_black_oxide"/>
@@ -139,5 +139,5 @@
     <origin xyz="0.091 -0.01275 -0.08725" rpy="0 0 0"/>
     <geometry>
-      <mesh filename="package://animatronics_urdf_description/meshes/XM,H,D-540.N101.I101_v5_1.stl" scale="0.001 0.001 0.001"/>
+      <mesh filename="package://animatronics_urdf_description/meshes/XM_H_D_540_N101_I101_v5_1.stl" scale="0.001 0.001 0.001"/>
     </geometry>
   </collision>
@@ -163,5 +163,5 @@
   </collision>
 </link>
-<link name="XM,H,D-540.N101.I101_v5_2">
+<link name="XM_H_D_540_N101_I101_v5_2">
   <inertial>
     <origin xyz="0.011512563950167629 -0.00966018872410861 -0.023818331012862903" rpy="0 0 0"/>
@@ -172,5 +172,5 @@
     <origin xyz="0.099 -0.03725 -0.1545" rpy="0 0 0"/>
     <geometry>
-      <mesh filename="package://animatronics_urdf_description/meshes/XM,H,D-540.N101.I101_v5_2.stl" scale="0.001 0.001 0.001"/>
+      <mesh filename="package://animatronics_urdf_description/meshes/XM_H_D_540_N101_I101_v5_2.stl" scale="0.001 0.001 0.001"/>
     </geometry>
     <material name="coating_black_oxide"/>
@@ -179,5 +179,5 @@
     <origin xyz="0.099 -0.03725 -0.1545" rpy="0 0 0"/>
     <geometry>
-      <mesh filename="package://animatronics_urdf_description/meshes/XM,H,D-540.N101.I101_v5_2.stl" scale="0.001 0.001 0.001"/>
+      <mesh filename="package://animatronics_urdf_description/meshes/XM_H_D_540_N101_I101_v5_2.stl" scale="0.001 0.001 0.001"/>
     </geometry>
   </collision>
@@ -203,5 +203,5 @@
   </collision>
 </link>
-<link name="XM,H,D-540.N101.I101_v5_3">
+<link name="XM_H_D_540_N101_I101_v5_3">
   <inertial>
     <origin xyz="0.006830257227709316 -0.02759715226246829 -0.007318331012862944" rpy="0 0 0"/>
@@ -212,5 +212,5 @@
     <origin xyz="-0.034717 0.053086 -0.138" rpy="0 0 0"/>
     <geometry>
-      <mesh filename="package://animatronics_urdf_description/meshes/XM,H,D-540.N101.I101_v5_3.stl" scale="0.001 0.001 0.001"/>
+      <mesh filename="package://animatronics_urdf_description/meshes/XM_H_D_540_N101_I101_v5_3.stl" scale="0.001 0.001 0.001"/>
     </geometry>
     <material name="coating_black_oxide"/>
@@ -219,5 +219,5 @@
     <origin xyz="-0.034717 0.053086 -0.138" rpy="0 0 0"/>
     <geometry>
-      <mesh filename="package://animatronics_urdf_description/meshes/XM,H,D-540.N101.I101_v5_3.stl" scale="0.001 0.001 0.001"/>
+      <mesh filename="package://animatronics_urdf_description/meshes/XM_H_D_540_N101_I101_v5_3.stl" scale="0.001 0.001 0.001"/>
     </geometry>
   </collision>
@@ -243,5 +243,5 @@
   </collision>
 </link>
-<link name="XM,H,D-540.N101.I101_v5_4">
+<link name="XM_H_D_540_N101_I101_v5_4">
   <inertial>
     <origin xyz="0.008620350868605839 -0.01231037038971286 -0.023818331012862903" rpy="0 0 0"/>
@@ -252,5 +252,5 @@
     <origin xyz="0.024075 0.182269 -0.1545" rpy="0 0 0"/>
     <geometry>
-      <mesh filename="package://animatronics_urdf_description/meshes/XM,H,D-540.N101.I101_v5_4.stl" scale="0.001 0.001 0.001"/>
+      <mesh filename="package://animatronics_urdf_description/meshes/XM_H_D_540_N101_I101_v5_4.stl" scale="0.001 0.001 0.001"/>
     </geometry>
     <material name="coating_black_oxide"/>
@@ -259,5 +259,5 @@
     <origin xyz="0.024075 0.182269 -0.1545" rpy="0 0 0"/>
     <geometry>
-      <mesh filename="package://animatronics_urdf_description/meshes/XM,H,D-540.N101.I101_v5_4.stl" scale="0.001 0.001 0.001"/>
+      <mesh filename="package://animatronics_urdf_description/meshes/XM_H_D_540_N101_I101_v5_4.stl" scale="0.001 0.001 0.001"/>
     </geometry>
   </collision>
@@ -323,5 +323,5 @@
   </collision>
 </link>
-<link name="XM,H,D-540.N101.I101_v5_5">
+<link name="XM_H_D_540_N101_I101_v5_5">
   <inertial>
     <origin xyz="-0.00731833202934741 0.022971414590661272 -0.01675000001560286" rpy="0 0 0"/>
@@ -332,5 +332,5 @@
     <origin xyz="0.091 -0.01275 0.05375" rpy="0 0 0"/>
     <geometry>
-      <mesh filename="package://animatronics_urdf_description/meshes/XM,H,D-540.N101.I101_v5_5.stl" scale="0.001 0.001 0.001"/>
+      <mesh filename="package://animatronics_urdf_description/meshes/XM_H_D_540_N101_I101_v5_5.stl" scale="0.001 0.001 0.001"/>
     </geometry>
     <material name="coating_black_oxide"/>
@@ -339,5 +339,5 @@
     <origin xyz="0.091 -0.01275 0.05375" rpy="0 0 0"/>
     <geometry>
-      <mesh filename="package://animatronics_urdf_description/meshes/XM,H,D-540.N101.I101_v5_5.stl" scale="0.001 0.001 0.001"/>
+      <mesh filename="package://animatronics_urdf_description/meshes/XM_H_D_540_N101_I101_v5_5.stl" scale="0.001 0.001 0.001"/>
     </geometry>
   </collision>
@@ -363,5 +363,5 @@
   </collision>
 </link>
-<link name="XM,H,D-540.N101.I101_v5_6">
+<link name="XM_H_D_540_N101_I101_v5_6">
   <inertial>
     <origin xyz="0.011512563818134189 -0.009660188678067227 0.02381833100689157" rpy="0 0 0"/>
@@ -372,5 +372,5 @@
     <origin xyz="0.099 -0.03725 0.1545" rpy="0 0 0"/>
     <geometry>
-      <mesh filename="package://animatronics_urdf_description/meshes/XM,H,D-540.N101.I101_v5_6.stl" scale="0.001 0.001 0.001"/>
+      <mesh filename="package://animatronics_urdf_description/meshes/XM_H_D_540_N101_I101_v5_6.stl" scale="0.001 0.001 0.001"/>
     </geometry>
     <material name="coating_black_oxide"/>
@@ -379,5 +379,5 @@
     <origin xyz="0.099 -0.03725 0.1545" rpy="0 0 0"/>
     <geometry>
-      <mesh filename="package://animatronics_urdf_description/meshes/XM,H,D-540.N101.I101_v5_6.stl" scale="0.001 0.001 0.001"/>
+      <mesh filename="package://animatronics_urdf_description/meshes/XM_H_D_540_N101_I101_v5_6.stl" scale="0.001 0.001 0.001"/>
     </geometry>
   </collision>
@@ -403,5 +403,5 @@
   </collision>
 </link>
-<link name="XM,H,D-540.N101.I101_v5_7">
+<link name="XM_H_D_540_N101_I101_v5_7">
   <inertial>
     <origin xyz="0.02836425709577542 -0.0019341522163085073 -0.008681668993108432" rpy="0 0 0"/>
@@ -412,5 +412,5 @@
     <origin xyz="-0.013183 0.078749 0.122" rpy="0 0 0"/>
     <geometry>
-      <mesh filename="package://animatronics_urdf_description/meshes/XM,H,D-540.N101.I101_v5_7.stl" scale="0.001 0.001 0.001"/>
+      <mesh filename="package://animatronics_urdf_description/meshes/XM_H_D_540_N101_I101_v5_7.stl" scale="0.001 0.001 0.001"/>
     </geometry>
     <material name="coating_black_oxide"/>
@@ -419,5 +419,5 @@
     <origin xyz="-0.013183 0.078749 0.122" rpy="0 0 0"/>
     <geometry>
-      <mesh filename="package://animatronics_urdf_description/meshes/XM,H,D-540.N101.I101_v5_7.stl" scale="0.001 0.001 0.001"/>
+      <mesh filename="package://animatronics_urdf_description/meshes/XM_H_D_540_N101_I101_v5_7.stl" scale="0.001 0.001 0.001"/>
     </geometry>
   </collision>
@@ -443,5 +443,5 @@
   </collision>
 </link>
-<link name="XM,H,D-540.N101.I101_v5_8">
+<link name="XM_H_D_540_N101_I101_v5_8">
   <inertial>
     <origin xyz="0.00862035073655892 -0.012310370343656785 0.023818331006891513" rpy="0 0 0"/>
@@ -452,5 +452,5 @@
     <origin xyz="0.024075 0.182269 0.1545" rpy="0 0 0"/>
     <geometry>
-      <mesh filename="package://animatronics_urdf_description/meshes/XM,H,D-540.N101.I101_v5_8.stl" scale="0.001 0.001 0.001"/>
+      <mesh filename="package://animatronics_urdf_description/meshes/XM_H_D_540_N101_I101_v5_8.stl" scale="0.001 0.001 0.001"/>
     </geometry>
     <material name="coating_black_oxide"/>
@@ -459,5 +459,5 @@
     <origin xyz="0.024075 0.182269 0.1545" rpy="0 0 0"/>
     <geometry>
-      <mesh filename="package://animatronics_urdf_description/meshes/XM,H,D-540.N101.I101_v5_8.stl" scale="0.001 0.001 0.001"/>
+      <mesh filename="package://animatronics_urdf_description/meshes/XM_H_D_540_N101_I101_v5_8.stl" scale="0.001 0.001 0.001"/>
     </geometry>
   </collision>
@@ -523,5 +523,5 @@
   </collision>
 </link>
-<link name="XM,H-430_idler_v3_1">
+<link name="XM_H_430_idler_v3_1">
   <inertial>
     <origin xyz="-0.019683702260469157 0.011000000128979462 0.017067018759162545" rpy="0 0 0"/>
@@ -532,5 +532,5 @@
     <origin xyz="-0.117 -0.00325 0.0215" rpy="0 0 0"/>
     <geometry>
-      <mesh filename="package://animatronics_urdf_description/meshes/XM,H-430_idler_v3_1.stl" scale="0.001 0.001 0.001"/>
+      <mesh filename="package://animatronics_urdf_description/meshes/XM_H_430_idler_v3_1.stl" scale="0.001 0.001 0.001"/>
     </geometry>
     <material name="steel_satin"/>
@@ -539,5 +539,5 @@
     <origin xyz="-0.117 -0.00325 0.0215" rpy="0 0 0"/>
     <geometry>
-      <mesh filename="package://animatronics_urdf_description/meshes/XM,H-430_idler_v3_1.stl" scale="0.001 0.001 0.001"/>
+      <mesh filename="package://animatronics_urdf_description/meshes/XM_H_430_idler_v3_1.stl" scale="0.001 0.001 0.001"/>
     </geometry>
   </collision>
@@ -603,5 +603,5 @@
   </collision>
 </link>
-<link name="6900ZZNR_v2_2">
+<link name="Link_6900ZZNR_v2_2">
   <inertial>
     <origin xyz="6.693118281830834e-13 6.320638457069094e-14 -0.003000000017362319" rpy="0 0 0"/>
@@ -612,5 +612,5 @@
     <origin xyz="-0.11025 -0.05575 0.0155" rpy="0 0 0"/>
     <geometry>
-      <mesh filename="package://animatronics_urdf_description/meshes/6900ZZNR_v2_2.stl" scale="0.001 0.001 0.001"/>
+      <mesh filename="package://animatronics_urdf_description/meshes/Link_6900ZZNR_v2_2.stl" scale="0.001 0.001 0.001"/>
     </geometry>
     <material name="steel_satin"/>
@@ -619,9 +619,9 @@
     <origin xyz="-0.11025 -0.05575 0.0155" rpy="0 0 0"/>
     <geometry>
-      <mesh filename="package://animatronics_urdf_description/meshes/6900ZZNR_v2_2.stl" scale="0.001 0.001 0.001"/>
-    </geometry>
-  </collision>
-</link>
-<link name="6900ZZNR_v2_1">
+      <mesh filename="package://animatronics_urdf_description/meshes/Link_6900ZZNR_v2_2.stl" scale="0.001 0.001 0.001"/>
+    </geometry>
+  </collision>
+</link>
+<link name="Link_6900ZZNR_v2_1">
   <inertial>
     <origin xyz="6.209616154606579e-13 5.796058077933708e-14 -0.0030000000173622567" rpy="0 0 0"/>
@@ -632,5 +632,5 @@
     <origin xyz="-0.11025 -0.05575 -0.0215" rpy="0 0 0"/>
     <geometry>
-      <mesh filename="package://animatronics_urdf_description/meshes/6900ZZNR_v2_1.stl" scale="0.001 0.001 0.001"/>
+      <mesh filename="package://animatronics_urdf_description/meshes/Link_6900ZZNR_v2_1.stl" scale="0.001 0.001 0.001"/>
     </geometry>
     <material name="steel_satin"/>
@@ -639,9 +639,9 @@
     <origin xyz="-0.11025 -0.05575 -0.0215" rpy="0 0 0"/>
     <geometry>
-      <mesh filename="package://animatronics_urdf_description/meshes/6900ZZNR_v2_1.stl" scale="0.001 0.001 0.001"/>
-    </geometry>
-  </collision>
-</link>
-<link name="XL-430_new_v5_1">
+      <mesh filename="package://animatronics_urdf_description/meshes/Link_6900ZZNR_v2_1.stl" scale="0.001 0.001 0.001"/>
+    </geometry>
+  </collision>
+</link>
+<link name="XL_430_new_v5_1">
   <inertial>
     <origin xyz="-0.006210633295508319 0.025330786091814946 0.011008281617777189" rpy="0 0 0"/>
@@ -652,5 +652,5 @@
     <origin xyz="-0.130949 -0.059914 0.011099" rpy="0 0 0"/>
     <geometry>
-      <mesh filename="package://animatronics_urdf_description/meshes/XL-430_new_v5_1.stl" scale="0.001 0.001 0.001"/>
+      <mesh filename="package://animatronics_urdf_description/meshes/XL_430_new_v5_1.stl" scale="0.001 0.001 0.001"/>
     </geometry>
     <material name="silver_default"/>
@@ -659,5 +659,5 @@
     <origin xyz="-0.130949 -0.059914 0.011099" rpy="0 0 0"/>
     <geometry>
-      <mesh filename="package://animatronics_urdf_description/meshes/XL-430_new_v5_1.stl" scale="0.001 0.001 0.001"/>
+      <mesh filename="package://animatronics_urdf_description/meshes/XL_430_new_v5_1.stl" scale="0.001 0.001 0.001"/>
     </geometry>
   </collision>
@@ -743,5 +743,5 @@
   </collision>
 </link>
-<link name="2XC-430_v6_1">
+<link name="Link_2XC_430_v6_1">
   <inertial>
     <origin xyz="3.8730834067995934e-05 0.012000459371747318 -0.019038679827954846" rpy="0 0 0"/>
@@ -752,5 +752,5 @@
     <origin xyz="-0.157104 -0.156228 -0.018801" rpy="0 0 0"/>
     <geometry>
-      <mesh filename="package://animatronics_urdf_description/meshes/2XC-430_v6_1.stl" scale="0.001 0.001 0.001"/>
+      <mesh filename="package://animatronics_urdf_description/meshes/Link_2XC_430_v6_1.stl" scale="0.001 0.001 0.001"/>
     </geometry>
     <material name="steel_satin"/>
@@ -759,5 +759,5 @@
     <origin xyz="-0.157104 -0.156228 -0.018801" rpy="0 0 0"/>
     <geometry>
-      <mesh filename="package://animatronics_urdf_description/meshes/2XC-430_v6_1.stl" scale="0.001 0.001 0.001"/>
+      <mesh filename="package://animatronics_urdf_description/meshes/Link_2XC_430_v6_1.stl" scale="0.001 0.001 0.001"/>
     </geometry>
   </collision>
@@ -803,5 +803,5 @@
   </collision>
 </link>
-<link name="XL-430_new_v5_2">
+<link name="XL_430_new_v5_2">
   <inertial>
     <origin xyz="0.020332416006495213 -0.011007747728442957 -0.017665721643406695" rpy="0 0 0"/>
@@ -812,5 +812,5 @@
     <origin xyz="-0.180604 -0.156728 -0.016801" rpy="0 0 0"/>
     <geometry>
-      <mesh filename="package://animatronics_urdf_description/meshes/XL-430_new_v5_2.stl" scale="0.001 0.001 0.001"/>
+      <mesh filename="package://animatronics_urdf_description/meshes/XL_430_new_v5_2.stl" scale="0.001 0.001 0.001"/>
     </geometry>
     <material name="silver_default"/>
@@ -819,5 +819,5 @@
     <origin xyz="-0.180604 -0.156728 -0.016801" rpy="0 0 0"/>
     <geometry>
-      <mesh filename="package://animatronics_urdf_description/meshes/XL-430_new_v5_2.stl" scale="0.001 0.001 0.001"/>
+      <mesh filename="package://animatronics_urdf_description/meshes/XL_430_new_v5_2.stl" scale="0.001 0.001 0.001"/>
     </geometry>
   </collision>
@@ -883,5 +883,5 @@
   </collision>
 </link>
-<link name="51202_v2_5">
+<link name="Link_51202_v2_5">
   <inertial>
     <origin xyz="-2.674484245179798e-10 0.0059999999999999915 9.592826533122434e-12" rpy="0 0 0"/>
@@ -892,5 +892,5 @@
     <origin xyz="0.099 -0.0685 -0.0705" rpy="0 0 0"/>
     <geometry>
-      <mesh filename="package://animatronics_urdf_description/meshes/51202_v2_5.stl" scale="0.001 0.001 0.001"/>
+      <mesh filename="package://animatronics_urdf_description/meshes/Link_51202_v2_5.stl" scale="0.001 0.001 0.001"/>
     </geometry>
     <material name="steel_satin"/>
@@ -899,5 +899,5 @@
     <origin xyz="0.099 -0.0685 -0.0705" rpy="0 0 0"/>
     <geometry>
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